File: engineering/electronics/pcbs/CBC_PCB/kicad/POWER SECTION.kicad_sch (KiCad schematic)
At the start: 72 parts, among them J4 AMT0650009DB0000G, J5 AMT0650009DB0000G, J6 AMT0650009DB0000G, J7 AMT0650009DB0000G, Q4 SP015N03BGHTO, U10 CPC1106NTR, U11 CPC1106NTR, U12 74LVC1G17W5-7, U13 74LVC2G02HK3-7, U14 MAX810R, U15 XL7056E1, U16 1kΩ, U17 1kΩ, U18 1kΩ, U19 1kΩ, U20 1kΩ, U21 1kΩ, U22 CPC1019NTR, U31 1kΩ, U32 1kΩ

Commit message: fix: restore CBC schematic library nicknames
Parts:
- C27, C28, C31: symbol CBC_PCB:GRM21BR61H106KE43L -> EasyEDA_Lib:GRM21BR61H106KE43L
- C29, C34: symbol CBC_PCB:LKME1252A101MF -> EasyEDA_Lib:LKME1252A101MF
- C30, C32, C33: symbol CBC_PCB:CL10B104KC8NNNC -> EasyEDA_Lib:CL10B104KC8NNNC
- CN2: symbol CBC_PCB:A1257WV-S-2P -> EasyEDA_Lib:A1257WV-S-2P
- D10, D11, D12, D13, D22, D23, D6, D8: symbol CBC_PCB:SMBJ13CA_C19077568 -> EasyEDA_Lib:SMBJ13CA_C19077568
- D5: symbol CBC_PCB:FSV10150V -> EasyEDA_Lib:FSV10150V
- D7: symbol CBC_PCB:SMBJ78CA_C2903953 -> EasyEDA_Lib:SMBJ78CA_C2903953
- D9: symbol CBC_PCB:ES3D_C241735 -> EasyEDA_Lib:ES3D_C241735
- F1: symbol CBC_PCB:0154005.DR -> EasyEDA_Lib:0154005.DR
- HC1, HC3: symbol CBC_PCB:C90D_PAD -> C90D_PAD:C90D_PAD
- J4, J5, J6, J7: symbol CBC_PCB:AMT0650009DB0000G -> AMT0650009DB0000G:AMT0650009DB0000G
- L3: symbol CBC_PCB:SMMS0650-101M -> EasyEDA_Lib:SMMS0650-101M
- Q10, Q11, Q2, Q3, Q4, Q5, Q6, Q7: symbol CBC_PCB:SP015N03BGHTO -> EasyEDA_Lib:SP015N03BGHTO
- R12, R16, R20, R24, R25, R26, R27, R28, R46, R47: symbol CBC_PCB:RT0402BRD0710KL -> EasyEDA_Lib:RT0402BRD0710KL
- R13: symbol CBC_PCB:RT0603BRD07100KL -> EasyEDA_Lib:RT0603BRD07100KL
- R14: symbol CBC_PCB:RT0402BRD073K3L -> EasyEDA_Lib:RT0402BRD073K3L
- R15, R23, R29: symbol CBC_PCB:RC0402FR-07330RL -> EasyEDA_Lib:RC0402FR-07330RL
- R17: symbol CBC_PCB:RT0603BRD072K7L -> EasyEDA_Lib:RT0603BRD072K7L
- R18: symbol CBC_PCB:0603WAF2372T5E -> EasyEDA_Lib:0603WAF2372T5E
- R19: symbol CBC_PCB:JER1206F1R060 -> EasyEDA_Lib:JER1206F1R060
- R21, R22: symbol CBC_PCB:AC05000003309JAC00 -> EasyEDA_Lib:AC05000003309JAC00
- R48: symbol CBC_PCB:25121WF100JT4E -> EasyEDA_Lib:25121WF100JT4E
- U10, U11: symbol CBC_PCB:CPC1106NTR -> EasyEDA_Lib:CPC1106NTR
- U12: symbol CBC_PCB:74LVC1G17W5-7 -> EasyEDA_Lib:74LVC1G17W5-7
- U13: symbol CBC_PCB:74LVC2G02HK3-7 -> EasyEDA_Lib:74LVC2G02HK3-7
- U14: symbol CBC_PCB:MAX810R -> EasyEDA_Lib:MAX810R
- U15: symbol CBC_PCB:XL7056E1 -> EasyEDA_Lib:XL7056E1
- U16, U17, U18, U19, U20, U21, U31, U32: symbol CBC_PCB:MCS0402MC1001FE000 -> EasyEDA_Lib:MCS0402MC1001FE000
- U22: symbol CBC_PCB:CPC1019NTR -> EasyEDA_Lib:CPC1019NTR
Connections:
- net +3V3: now also C28.2, C31.2, U12.5 (VCC), U13.8 (VCC), U14.3 (VCC)
- net 12V_GATE_V: now also R18.2, R19.2, U11.4 (Load), U15.5 (CSP), U22.4
- net 12V_TRIGGER_SIG: now also R13.1
- net CANH_BAT: now also CN2.1
- net CANL_BAT: now also CN2.2
- net ESP_ENABLE_SIGNAL: now also R16.2, U13.1 (1A)
- net GND: now also C27.1, C28.1, C31.1, D7.2, J7.1, J7.2, J7.3, J7.4, J7.5, J7.6, Q10.9 (D), Q11.9 (D), Q3.9 (D), Q4.9 (D), Q5.9 (D), Q6.9 (D), Q7.9 (D), R14.1, R16.1, R21.2, R22.2, U10.2 (-Control), U11.2 (-Control), U12.3 (GND), U13.4 (GND), U14.1 (GND), U22.2
- net H_PWR-IN: now also D9.1, HC1.1, J6.1, J6.2, J6.3, J6.4, J6.5, J6.6, R48.2
- net H_PWR-IN-: now also C29.2, C30.1, C33.1, C34.2, D10.1, D11.1, D12.1, D13.1, D22.1, D23.1, D5.1 (A), D5.2 (A), D6.1, D7.1, D8.1, F1.1, J5.1, J5.2, J5.3, J5.4, J5.5, J5.6, Q10.2 (S), Q10.3 (S), Q10.4 (S), Q10.5 (S), Q10.6 (S), Q10.7 (S), Q10.8 (S), Q11.2 (S), Q11.3 (S), Q11.4 (S), Q11.5 (S), Q11.6 (S), Q11.7 (S), Q11.8 (S), Q3.2 (S), Q3.3 (S), Q3.4 (S), Q3.5 (S), Q3.6 (S), Q3.7 (S), Q3.8 (S), Q4.2 (S), Q4.3 (S), Q4.4 (S), Q4.5 (S), Q4.6 (S), Q4.7 (S), Q4.8 (S), Q5.2 (S), Q5.3 (S), Q5.4 (S), Q5.5 (S), Q5.6 (S), Q5.7 (S), Q5.8 (S), Q6.2 (S), Q6.3 (S), Q6.4 (S), Q6.5 (S), Q6.6 (S), Q6.7 (S), Q6.8 (S), Q7.2 (S), Q7.3 (S), Q7.4 (S), Q7.5 (S), Q7.6 (S), Q7.7 (S), Q7.8 (S), R17.1, R20.1, R24.1, R25.1, R26.1, R27.1, R28.1, R46.1, R47.1, U15.1 (GND), U15.8 (EP)
- net H_PWR-IN--PREFUSE: now also HC3.1, J4.1, J4.2, J4.3, J4.4, J4.5, J4.6
- net MOSFET_CONTROL_SIGNAL: now also R29.2, U10.4 (Load)
- net OUTPUT: now also C27.2, R12.2, R13.2
- net PRECHARGE_ESP_SIGNAL: now also R23.2
- net SCHMITT_OUT: now also R15.2, U12.4 (Y)
- net STARTUP_RESET: now also U13.6 (2B), U14.2 (RESET#)
- net SWITCHED_GATE_V: now also U17.2, U18.2, U19.2, U20.2, U21.2, U22.3, U31.2, U32.2
- new net: R12.1, R14.2, U12.2 (A)
- new net: F1.2, Q2.2 (S), Q2.3 (S), Q2.4 (S), Q2.5 (S), Q2.6 (S), Q2.7 (S), Q2.8 (S)
- new net: D8.2, Q3.1 (G), R24.2, U17.1
- new net: D5.3 (K), L3.1, U15.4 (SW)
- new net: C33.2, C34.1, L3.2, R19.1, U15.3 (CSN)
- new net: D13.2, Q7.1 (G), R28.2, U21.1
- new net: D10.2, Q4.1 (G), R25.2, U18.1
- new net: R15.1, U10.1 (+Control)
- new net: U10.3 (Load), U13.2 (1B), U13.3 (2Y)
- new net: D22.2, Q10.1 (G), R46.2, U31.1
- new net: C29.1, C30.2, C32.1, R48.1, U15.7 (VIN)
- new net: D6.2, Q2.1 (G), R20.2, U16.1
- new net: D9.2, Q2.9 (D), R21.1, R22.1
- new net: R29.1, U22.1
- new net: D12.2, Q6.1 (G), R27.2, U20.1
- new net: D11.2, Q5.1 (G), R26.2, U19.1
- new net: C32.2, U15.6 (VC)
- new net: R17.2, R18.1, U15.2 (FB)
- new net: D23.2, Q11.1 (G), R47.2, U32.1
- new net: U11.3 (Load), U16.2
- new net: R23.1, U11.1 (+Control)
- new net: U13.5 (2A), U13.7 (1Y)

Commit message: fix: qualify CBC connector footprint refs
Parts:
- J4, J5, J6, J7: footprint AMT0650009DB0000G -> CBC_PCB:AMT0650009DB0000G
