File: engineering/electronics/pcbs/CBC_PCB/kicad/CBC_PCB.kicad_pcb (KiCad board)
At the start: 6 copper layers, 178 x 211 mm, 285 parts, among them J2 AT13-12PB-BM03, J4 AMT0650009DB0000G, J5 AMT0650009DB0000G, J6 AMT0650009DB0000G, J7 AMT0650009DB0000G, Q4 SP015N03BGHTO, U10 CPC1106NTR, U11 CPC1106NTR, U12 74LVC1G17W5-7, U13 74LVC2G02HK3-7, U14 MAX810R, U15 MAX40203AUK+T, U16 1kΩ, U17 1kΩ, U18 1kΩ, U19 1kΩ, U2 2.4GHz, U20 1kΩ, U21 1kΩ, U22 CPC1019NTR, U23 MP9486GN-Z, U25 ADM3053BRWZ-REEL7, U26 ADM3053BRWZ-REEL7, U27 10mΩ, U29 1uF, U30 1uH, U31 1kΩ, U32 1kΩ, U33 MP9486GN-Z, U34 MP9486GN-Z, U35 MP9486GN-Z, U37 MAX40203AUK+T, U38 MAX40203AUK+T, U39 MAX40203AUK+T, U9 120pF, X1 16MHz, X2 16MHz

Commit message: electronics: integrate CBC PCB footprint updates
Parts:
- moved R15 130.9 mm to (107.5, 179.2)
- moved R29 130.9 mm to (106.8, 184.9)
- moved U10 130.9 mm to (112.0, 178.8)
- moved U13 130.9 mm to (118.7, 183.3)
- moved U22 130.9 mm to (112.0, 186.2)
- moved C31 130.9 mm to (121.3, 182.7)
- moved U14 130.9 mm to (119.3, 186.9)
- moved R16 129.6 mm to (119.5, 179.7)
- moved R58 3.45 mm to (110.6, 123.6)
- moved R59 3.39 mm to (110.6, 120.1)
- moved C11 3.26 mm to (109.5, 224.2)
- moved D20 2.67 mm to (156.6, 205.3)
- moved C45 2.39 mm to (80.7, 136.7)
- moved C46 2.39 mm to (83.6, 135.7)
- moved U24 2.39 mm to (75.0, 136.0)
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Connections:
- R62 pad 1: +5V_P2 -> +3V3_P2
- U39 pad 1: +5V_P2 -> +3V3_P2
Routing:
- net +3V3: track 229.0 -> 560.9 mm, vias 9 -> 11
- net H_PWR-IN-: track 0.00 -> 254.4 mm, vias 1 -> 4
- net H_PWR-IN: track 87.1 -> 329.5 mm, vias 3 -> 4
- net 12V_GATE_V: track 1.59 -> 222.4 mm, vias 1 -> 3
- net /CAN SECTION/TXD: track 3.49 -> 209.2 mm
- net +5V: track 94.4 -> 300.1 mm, vias 3 -> 8
- net /CAN SECTION/RXD: track 5.61 -> 206.7 mm
- net PRECHARGE_ESP_SIGNAL: track 29.3 -> 207.7 mm, vias 2 -> 0
- net TEMP1_DQ: track 8.33 -> 161.2 mm, vias 1 -> 2
- net /POWER SECTION/SWITCHED_GATE_V: track 92.8 -> 213.3 mm, vias 0 -> 3
- net 12V_TRIGGER_SIG: track 0.00 -> 52.9 mm, vias 0 -> 2
- net SCHMITT_OUT: track 25.1 -> 72.4 mm, vias 5 -> 2
- net CANL_DRONE: track 12.6 -> 57.2 mm
- net ESP_ENABLE_SIGNAL: track 31.4 -> 74.4 mm
- net GND_CB: track 45.6 -> 87.9 mm, vias 2 -> 3
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- added copper zone on In2.Cu, net GNDE
- added copper zone on In3.Cu, net GNDE
- removed copper zone on B.Cu, net GNDE
Other:
- board text removed: "- HC1 and HC3 need to stay in that location - Screw terminals should also be in that general are - If Mosfets are moved, please take note of the two mounting holes left and right from the mosfets. Distance should be 100mm. - Output connector should be in the bottom middle section of the PCB. - Everything else can be moved around if necessary."

Commit message: electronics: fix CBC footprint component types
Parts:
- moved C14 2.28 mm to (98.0, 227.5), turned to 0 degrees
Routing:
- net H_PWR-IN: track 329.5 -> 335.1 mm
- net +5V: track 300.1 -> 303.1 mm
- net +3V3: track 560.9 -> 562.7 mm
- net PRECHARGE_ESP_SIGNAL: track 207.7 -> 209.1 mm
- added copper zone on B.Cu, net GND_CA
- added copper zone on In2.Cu, net Net-(C66-Pad2)
- added copper zone on In3.Cu, net Net-(C66-Pad2)
- added copper zone on In2.Cu, net Net-(C71-Pad2)
- added copper zone on In3.Cu, net Net-(C71-Pad2)
- added copper zone on In2.Cu, net Net-(D19-A)
- added copper zone on In3.Cu, net Net-(D19-A)
- removed copper zone on In2.Cu, net GND_CA
- removed copper zone on B.Cu, net Net-(C66-Pad2)
- removed copper zone on B.Cu, net Net-(C71-Pad2)
- removed copper zone on B.Cu, net Net-(D19-A)
- removed copper zone on B.Cu, net Net-(Q2-D)
- removed copper zone on In1.Cu, net Net-(Q2-D)
- removed copper zone on In4.Cu, net Net-(Q2-D)
Other:
- outline, holes or cut-outs redrawn
