File: engineering/electronics/pcbs/CBC_PCB/kicad/POWER REGULATOR.kicad_sch (KiCad schematic)
At the start: 107 parts, among them U15 MAX40203AUK+T, U23 MP9486GN-Z, U27 10mΩ, U29 1uF, U30 1uH, U35 MP9486GN-Z, U37 MAX40203AUK+T, U38 MAX40203AUK+T, U39 MAX40203AUK+T, U9 120pF

Commit message: pcb: update CBC import and routing rules
Parts:
- added C110, C111: 100nF, EasyEDA_Lib:C0603, symbol CBC_PCB:CL10B104KC8NNNC
- C37, C39, C75, C76, C93, C94: footprint EasyEDA_Lib:CAP-TH_BD5.0-P2.00-D0.5-FD-1 -> EasyEDA_Lib_2:C2220; symbol CBC_PCB:ERJ1KM2R2D11OT -> EasyEDA_Lib_2:FS55X225K251EGG; LCSC Part Name 2.2uF ±20% 100V -> 2.2uF ±10% 250V; Manufacturer AISHI(艾华集团) -> PSA(信昌电陶); Manufacturer Part ERJ1KM2R2D11OT -> FS55X225K251EGG; Supplier Part C694099 -> C153032
- C64: footprint EasyEDA_Lib:C1206 -> EasyEDA_Lib_2:CAP-SMD_BD10.0-L10.3-W10.3-FD-LS11.0; symbol CBC_PCB:GRM31CR61E476ME44L -> EasyEDA_Lib_2:EFPA100ADA470M10C0; LCSC Part Name 47uF ±20% 25V -> 47uF ±20% 100V; Manufacturer muRata(村田) -> FOLLON(富隆电子); Manufacturer Part GRM31CR61E476ME44L -> EFPA100ADA470M10C0; Supplier Part C403725 -> C49424130
- C65: footprint EasyEDA_Lib:C0603 -> EasyEDA_Lib_2:C0805; symbol CBC_PCB:CL10B333KB8NNNC -> EasyEDA_Lib_2:CC0805KKX7R0BB333; LCSC Part Name 33nF ±10% 50V -> 33nF ±10% 100V; Manufacturer SAMSUNG(三星) -> YAGEO(国巨); Manufacturer Part CL10B333KB8NNNC -> CC0805KKX7R0BB333; Supplier Part C21117 -> C327114
- D14, D28: footprint EasyEDA_Lib:TO-277A_L5.9-W4.4-LS6.5-TR -> EasyEDA_Lib_2:SMB_L4.6-W3.6-LS5.3-RD; symbol CBC_PCB:FSV10150V -> EasyEDA_Lib_2:SS3150/SMB; LCSC Part Name 电压:150V 电流:10A -> 电压:150V 电流:3A; Manufacturer onsemi(安森美) -> MDD(辰达半导体); Manufacturer Part FSV10150V -> SS3150B; Supplier Part C719814 -> C47124
- L4, L9: footprint EasyEDA_Lib:IND-SMD_L8.5-W8.0_SMS0850 -> EasyEDA_Lib_2:IND-SMD_L6.0-W6.0_SMNR6045; symbol CBC_PCB:ZEMS0850-330M -> EasyEDA_Lib_2:SMNR6045-330MT; LCSC Part Name 33UH ±20% 6A 一体成型电感，合金电感，大电流，低阻抗 -> 33uH ±20% 1.65A; Manufacturer ZE(增益) -> SXN(顺翔诺); Manufacturer Part ZEMS0850-330M -> SMNR6045-330MT; Supplier Part C41438711 -> C135306
- L6: footprint EasyEDA_Lib:IND-SMD_L11.0-W10.0-PSPMAA1082T -> EasyEDA_Lib_2:IND-SMD_L6.6-W6.4; symbol CBC_PCB:PSPMAA1082T-220M-CGP -> EasyEDA_Lib_2:XAL6060-223MEC; LCSC Part Name 22μH ±20% 13A -> 22uH ±20% 5.9A; Manufacturer PROD(谱罗德) -> Coilcraft(线艺); Manufacturer Part PSPMAA1082T-220M-CGP -> XAL6060-223MEC; Supplier Part C47149121 -> C5366013
- Q8: footprint EasyEDA_Lib:TOLL-8_L10.4-W9.9-P1.20-LS11.7-BL -> CBC_PCB:DFN-8_L5.9-W5.2-P1.27-LS6.2-BL; symbol CBC_PCB:SP015N03BGHTO -> CBC_PCB:BSC320N20NS3G; LCSC Part Name 耐压:150V 电流:260A -> 1个N沟道 耐压:200V 电流:36A; Manufacturer Siliup(矽普) -> Infineon(英飞凌); Manufacturer Part SP015N03BGHTO -> BSC320N20NS3G; Supplier Part C22385354 -> C501501
- Q9: footprint EasyEDA_Lib:TOLL-8_L10.4-W9.9-P1.20-LS11.7-BL -> CBC_PCB:DFN-8_L5.9-W5.2-P1.27-LS6.2-BL; symbol CBC_PCB:SP015N03BGHTO -> CBC_PCB:BSC047N08NS3G; LCSC Part Name 耐压:150V 电流:260A -> 1个N沟道 耐压:80V 电流:100A; Manufacturer Siliup(矽普) -> Infineon(英飞凌); Manufacturer Part SP015N03BGHTO -> BSC047N08NS3G; Supplier Part C22385354 -> C501500
- U62: renamed from C62; value 2.2uF -> 1uF; footprint EasyEDA_Lib:CAP-TH_BD5.0-P2.00-D0.5-FD-1 -> EasyEDA_Lib_2:C0805; symbol CBC_PCB:ERJ1KM2R2D11OT -> EasyEDA_Lib_2:CC0805KKX7R0BB105; LCSC Part Name 2.2uF ±20% 100V -> 1uF ±10% 100V; Manufacturer AISHI(艾华集团) -> YAGEO(国巨); Manufacturer Part ERJ1KM2R2D11OT -> CC0805KKX7R0BB105; Supplier Part C694099 -> C5370002
- renumbered U29 to C29
Connections:
- net GND: now also C37.1, C39.1, C64.2, C65.2, C93.1, C94.1, C110.2, C111.2; no longer C37.2, C39.2, C64.1, C65.1, C93.2, C94.2, D14.2 (A), D28.2 (A)
- net GNDE: now also C75.1, C76.1, Q9.1 (S); no longer C75.2, C76.2, Q9.2 (S), Q9.3 (S), Q9.4 (S), Q9.5 (S), Q9.6 (S), Q9.7 (S), Q9.8 (S)
- net H_PWR-IN: now also C37.2, C39.2, C64.1, C93.2, C94.2, C110.1, C111.1; no longer C37.1, C39.1, C64.2, C93.1, C94.1
- net at Q8.1 (S): now also R41.2, U27.2; no longer R36.2
- net at D18.2 (A), L5.1, L5.2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: now also Q8.3 (D); no longer Q8.9 (D)
- net at C41.1, L4.1, U23.5 (SW): now also D14.2 (K); no longer D14.3 (K)
- net at C71.2, C72.2, C77.2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: now also C75.2, C76.2; no longer C75.1, C76.1
- net at D19.2 (A), L5.7, L5.8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: now also Q9.3 (D); no longer Q9.9 (D)
- net at C95.1, L9.1, U35.5 (SW): now also D28.2 (K); no longer D28.3 (K)
- net at R42.1: now also C65.1; no longer C65.2
- net at U28.1 (GATE): now also Q9.2 (G); no longer Q9.1 (G)
- new net: Q8.2 (G), R36.2
Other:
- moved on the sheet: C65
