File: engineering/electronics/pcbs/CBC_PCB/kicad/POWER REGULATOR.kicad_sch (KiCad schematic)
At the start: 98 parts, among them U15 MAX40203AUK+T, U23 MP9486GN-Z, U27 10mΩ, U29 1uF, U30 1uH, U35 MP9486GN-Z, U37 MAX40203AUK+T, U38 MAX40203AUK+T, U39 MAX40203AUK+T, U9 120pF

Commit message: electronics: integrate CBC PCB updates
Parts:
- added F4, F5: (no value), EasyEDA_Lib:FUSE-SMD_L9.8-W5.1, symbol CBC_PCB:0154001.DR
- added F6: 0154005.DR, EasyEDA_Lib:FUSE-SMD_L9.8-W5.1, symbol CBC_PCB:0154005.DR
- added LED5, LED6, LED7: (no value), EasyEDA_Lib:LED0603-RD, symbol CBC_PCB:0603 Green 509-620mcd
- added R66, R67: 390Ω, EasyEDA_Lib:R0603, symbol CBC_PCB:0603WAF3900T5E
- added R68: 1.8kΩ, EasyEDA_Lib:R0603, symbol CBC_PCB:0603WAF1801T5E
- C100, C101, C103, C35, C41, C43, C44, C45, C95, C96: symbol EasyEDA_Lib:CL10B104KC8NNNC -> CBC_PCB:CL10B104KC8NNNC
- C102, C104, C42, C46: symbol EasyEDA_Lib:TAJB106K025RNJ -> CBC_PCB:TAJB106K025RNJ
- C15: symbol EasyEDA_Lib:CC0805KRX7R0BB471 -> CBC_PCB:CC0805KRX7R0BB471
- C37, C39, C62, C75, C76, C93, C94: symbol EasyEDA_Lib:ERJ1KM2R2D11OT -> CBC_PCB:ERJ1KM2R2D11OT
- C38, C40, C74, C97, C98, C99: symbol EasyEDA_Lib:CL21A475KBQNNNE -> CBC_PCB:CL21A475KBQNNNE
- C59, C60, C61, C7, C73: symbol EasyEDA_Lib:GRM31CC72A475KE11L -> CBC_PCB:GRM31CC72A475KE11L
- C63: symbol EasyEDA_Lib:CL10B224KB8NNNC -> CBC_PCB:CL10B224KB8NNNC
- C64, C66, C69, C70, C71, C72, C77: symbol EasyEDA_Lib:GRM31CR61E476ME44L -> CBC_PCB:GRM31CR61E476ME44L
- C65: symbol EasyEDA_Lib:CL10B333KB8NNNC -> CBC_PCB:CL10B333KB8NNNC
- C67: symbol EasyEDA_Lib:CL10C470JB8NNNC -> CBC_PCB:CL10C470JB8NNNC
- C68: symbol EasyEDA_Lib:AC0603KRX7R0BB472 -> CBC_PCB:AC0603KRX7R0BB472
- D14, D28: symbol EasyEDA_Lib:FSV10150V -> CBC_PCB:FSV10150V
- D15, D29: symbol EasyEDA_Lib:SMBJ5.0CA_C83323 -> CBC_PCB:SMBJ5.0CA_C83323
- D16, D19: symbol EasyEDA_Lib:BAV20W-7-F -> CBC_PCB:BAV20W-7-F
- D17: symbol EasyEDA_Lib:SMBJ85A-13-F -> CBC_PCB:SMBJ85A-13-F
- D18: symbol EasyEDA_Lib:CMMR1U-02 TR PBFREE -> CBC_PCB:CMMR1U-02 TR PBFREE
- D20: symbol EasyEDA_Lib:SMB5350B -> CBC_PCB:SMB5350B
- D21: symbol EasyEDA_Lib:SMBJ5365B-TP -> CBC_PCB:SMBJ5365B-TP
- L4, L9: symbol EasyEDA_Lib:ZEMS0850-330M -> CBC_PCB:ZEMS0850-330M
- L5: symbol EasyEDA_Lib:PA1736NL -> CBC_PCB:PA1736NL
- L6: symbol EasyEDA_Lib:PSPMAA1082T-220M-CGP -> CBC_PCB:PSPMAA1082T-220M-CGP
- Q8, Q9: symbol EasyEDA_Lib:SP015N03BGHTO -> CBC_PCB:SP015N03BGHTO
- R17, R18, R19, R5, R62: symbol EasyEDA_Lib:PTFR0603B100RN9 -> CBC_PCB:PTFR0603B100RN9
- R30, R33, R59, R61: symbol EasyEDA_Lib:RT0603BRD0710KL -> CBC_PCB:RT0603BRD0710KL
- R31, R58: symbol EasyEDA_Lib:RT0603BRE07240KL -> CBC_PCB:RT0603BRE07240KL
- R32, R60: symbol EasyEDA_Lib:PTFR0603B140KP9 -> CBC_PCB:PTFR0603B140KP9
- R36: symbol EasyEDA_Lib:RC0402FR-070RL -> CBC_PCB:RC0402FR-070RL
- R37: symbol EasyEDA_Lib:FRC0805F1204TS -> CBC_PCB:FRC0805F1204TS
- R38: symbol EasyEDA_Lib:PTFR0603B51K0P9 -> CBC_PCB:PTFR0603B51K0P9
- R39: symbol EasyEDA_Lib:0805W8F1603T5E -> CBC_PCB:0805W8F1603T5E
- R40: symbol EasyEDA_Lib:0603WAF6041T5E -> CBC_PCB:0603WAF6041T5E
- R41, R45: symbol EasyEDA_Lib:0805W8F300KT5E -> CBC_PCB:0805W8F300KT5E
- R42: symbol EasyEDA_Lib:FRC0603F7501TS -> CBC_PCB:FRC0603F7501TS
- R43: symbol EasyEDA_Lib:0603WAF6042T5E -> CBC_PCB:0603WAF6042T5E
- R44: symbol EasyEDA_Lib:FRC0603F2371TS -> CBC_PCB:FRC0603F2371TS
- R6: symbol EasyEDA_Lib:ERA6AEB680V -> CBC_PCB:ERA6AEB680V
- U15, U37, U38, U39: symbol EasyEDA_Lib:MAX40203AUK+T -> CBC_PCB:MAX40203AUK+T
- U23, U35: symbol MP9486GN-Z:MP9486GN-Z -> CBC_PCB:MP9486GN-Z
- U24, U36: symbol EasyEDA_Lib:AMS1117-3.3 -> CBC_PCB:AMS1117-3.3
- U27: symbol EasyEDA_Lib:YLRY06-1-10F -> CBC_PCB:YLRY06-1-10F
- U28: symbol EasyEDA_Lib:LT8309ES5#TRMPBF -> CBC_PCB:LT8309ES5#TRMPBF
- U29: symbol EasyEDA_Lib:CC0805KKX7R0BB105 -> CBC_PCB:CC0805KKX7R0BB105
- U30: symbol EasyEDA_Lib:XAL6030-102MEC -> CBC_PCB:XAL6030-102MEC
- U8: symbol EasyEDA_Lib:LT3748EMS#PBF -> CBC_PCB:LT3748EMS#PBF
- U9: symbol EasyEDA_Lib:GCM1885C2A121FA16D -> CBC_PCB:GCM1885C2A121FA16D
Connections:
- net +3V3: no longer C101.1, C102.1, C45.1, C46.1, U24.2 (VOUT), U36.2 (VOUT)
- net +3V3_P1: now also C45.1, C46.1, U24.2 (VOUT)
- net +3V3_P2: now also C101.1, C102.1, U36.2 (VOUT)
- net +5V_P1: now also F4.1; no longer R17.1, U15.1 (VDD)
- net +5V_P2: now also F5.1; no longer R18.1, U37.1 (VDD)
- net 12V_ISOLATED: now also F6.2, R68.2; no longer C71.2, C72.2, C75.1, C76.1, C77.2, D20.1, U30.2
- net GND: now also LED5.1 (K), LED6.1 (K)
- net GNDE: now also LED7.1 (K)
- new net: LED7.2 (A), R68.1
- new net: C71.2, C72.2, C75.1, C76.1, C77.2, D20.1, F6.1, U30.2
- new net: F5.2, R18.1, R67.1, U37.1 (VDD)
- new net: LED6.2 (A), R67.2
- new net: F4.2, R17.1, R66.1, U15.1 (VDD)
- new net: LED5.2 (A), R66.2

Commit message: electronics: integrate CBC PCB footprint updates
Connections:
- net +3V3_P2: now also R62.1, U39.1 (VDD)
- net +5V_P2: no longer R62.1, U39.1 (VDD)

Commit message: electronics: update CMAIN and CBC PCB files
Other:
- moved on the sheet: C15, C59, C60, C61, C62, C63, C64, C65, C66, C67, C68, C69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

Commit message: fix(cbc): integrate ordered PCB update
Parts:
- added C605, C606: 100nF, EasyEDA_Lib:C0603, symbol CBC_PCB:CL10B104KC8NNNC
- C601: renamed from C39; footprint EasyEDA_Lib:CAP-TH_BD5.0-P2.00-D0.5-FD-1 -> EasyEDA_Lib_2:C2220; symbol CBC_PCB:ERJ1KM2R2D11OT -> EasyEDA_Lib_2:FS55X225K251EGG; LCSC Part Name 2.2uF ±20% 100V -> 2.2uF ±10% 250V; Manufacturer AISHI(艾华集团) -> PSA(信昌电陶); Manufacturer Part ERJ1KM2R2D11OT -> FS55X225K251EGG; Supplier Part C694099 -> C153032
- C602: renamed from C93; footprint EasyEDA_Lib:CAP-TH_BD5.0-P2.00-D0.5-FD-1 -> EasyEDA_Lib_2:C2220; symbol CBC_PCB:ERJ1KM2R2D11OT -> EasyEDA_Lib_2:FS55X225K251EGG; LCSC Part Name 2.2uF ±20% 100V -> 2.2uF ±10% 250V; Manufacturer AISHI(艾华集团) -> PSA(信昌电陶); Manufacturer Part ERJ1KM2R2D11OT -> FS55X225K251EGG; Supplier Part C694099 -> C153032
- C603: renamed from C37; footprint EasyEDA_Lib:CAP-TH_BD5.0-P2.00-D0.5-FD-1 -> EasyEDA_Lib_2:C2220; symbol CBC_PCB:ERJ1KM2R2D11OT -> EasyEDA_Lib_2:FS55X225K251EGG; LCSC Part Name 2.2uF ±20% 100V -> 2.2uF ±10% 250V; Manufacturer AISHI(艾华集团) -> PSA(信昌电陶); Manufacturer Part ERJ1KM2R2D11OT -> FS55X225K251EGG; Supplier Part C694099 -> C153032
- C604: renamed from C94; footprint EasyEDA_Lib:CAP-TH_BD5.0-P2.00-D0.5-FD-1 -> EasyEDA_Lib_2:C2220; symbol CBC_PCB:ERJ1KM2R2D11OT -> EasyEDA_Lib_2:FS55X225K251EGG; LCSC Part Name 2.2uF ±20% 100V -> 2.2uF ±10% 250V; Manufacturer AISHI(艾华集团) -> PSA(信昌电陶); Manufacturer Part ERJ1KM2R2D11OT -> FS55X225K251EGG; Supplier Part C694099 -> C153032
- C609: renamed from C64; footprint EasyEDA_Lib:C1206 -> EasyEDA_Lib_2:CAP-SMD_BD10.0-L10.3-W10.3-FD-LS11.0; symbol CBC_PCB:GRM31CR61E476ME44L -> EasyEDA_Lib_2:EFPA100ADA470M10C0; LCSC Part Name 47uF ±20% 25V -> 47uF ±20% 100V; Manufacturer muRata(村田) -> FOLLON(富隆电子); Manufacturer Part GRM31CR61E476ME44L -> EFPA100ADA470M10C0; Supplier Part C403725 -> C49424130
- C613: renamed from C65; footprint EasyEDA_Lib:C0603 -> EasyEDA_Lib_2:C0805; symbol CBC_PCB:CL10B333KB8NNNC -> EasyEDA_Lib_2:CC0805KKX7R0BB333; LCSC Part Name 33nF ±10% 50V -> 33nF ±10% 100V; Manufacturer SAMSUNG(三星) -> YAGEO(国巨); Manufacturer Part CL10B333KB8NNNC -> CC0805KKX7R0BB333; Supplier Part C21117 -> C327114
- C644: renamed from C75; footprint EasyEDA_Lib:CAP-TH_BD5.0-P2.00-D0.5-FD-1 -> EasyEDA_Lib_2:C2220; symbol CBC_PCB:ERJ1KM2R2D11OT -> EasyEDA_Lib_2:FS55X225K251EGG; LCSC Part Name 2.2uF ±20% 100V -> 2.2uF ±10% 250V; Manufacturer AISHI(艾华集团) -> PSA(信昌电陶); Manufacturer Part ERJ1KM2R2D11OT -> FS55X225K251EGG; Supplier Part C694099 -> C153032
- C646: renamed from C76; footprint EasyEDA_Lib:CAP-TH_BD5.0-P2.00-D0.5-FD-1 -> EasyEDA_Lib_2:C2220; symbol CBC_PCB:ERJ1KM2R2D11OT -> EasyEDA_Lib_2:FS55X225K251EGG; LCSC Part Name 2.2uF ±20% 100V -> 2.2uF ±10% 250V; Manufacturer AISHI(艾华集团) -> PSA(信昌电陶); Manufacturer Part ERJ1KM2R2D11OT -> FS55X225K251EGG; Supplier Part C694099 -> C153032
- D601: renamed from D14; footprint EasyEDA_Lib:TO-277A_L5.9-W4.4-LS6.5-TR -> EasyEDA_Lib_2:SMB_L4.6-W3.6-LS5.3-RD; symbol CBC_PCB:FSV10150V -> EasyEDA_Lib_2:SS3150/SMB; LCSC Part Name 电压:150V 电流:10A -> 电压:150V 电流:3A; Manufacturer onsemi(安森美) -> MDD(辰达半导体); Manufacturer Part FSV10150V -> SS3150B; Supplier Part C719814 -> C47124
- D602: renamed from D28; footprint EasyEDA_Lib:TO-277A_L5.9-W4.4-LS6.5-TR -> EasyEDA_Lib_2:SMB_L4.6-W3.6-LS5.3-RD; symbol CBC_PCB:FSV10150V -> EasyEDA_Lib_2:SS3150/SMB; LCSC Part Name 电压:150V 电流:10A -> 电压:150V 电流:3A; Manufacturer onsemi(安森美) -> MDD(辰达半导体); Manufacturer Part FSV10150V -> SS3150B; Supplier Part C719814 -> C47124
- L601: renamed from L6; footprint EasyEDA_Lib:IND-SMD_L11.0-W10.0-PSPMAA1082T -> EasyEDA_Lib_2:IND-SMD_L6.6-W6.4; symbol CBC_PCB:PSPMAA1082T-220M-CGP -> EasyEDA_Lib_2:XAL6060-223MEC; LCSC Part Name 22μH ±20% 13A -> 22uH ±20% 5.9A; Manufacturer PROD(谱罗德) -> Coilcraft(线艺); Manufacturer Part PSPMAA1082T-220M-CGP -> XAL6060-223MEC; Supplier Part C47149121 -> C5366013
- L602: renamed from L4; footprint EasyEDA_Lib:IND-SMD_L8.5-W8.0_SMS0850 -> EasyEDA_Lib_2:IND-SMD_L6.0-W6.0_SMNR6045; symbol CBC_PCB:ZEMS0850-330M -> EasyEDA_Lib_2:SMNR6045-330MT; LCSC Part Name 33UH ±20% 6A 一体成型电感，合金电感，大电流，低阻抗 -> 33uH ±20% 1.65A; Manufacturer ZE(增益) -> SXN(顺翔诺); Manufacturer Part ZEMS0850-330M -> SMNR6045-330MT; Supplier Part C41438711 -> C135306
- L603: renamed from L9; footprint EasyEDA_Lib:IND-SMD_L8.5-W8.0_SMS0850 -> EasyEDA_Lib_2:IND-SMD_L6.0-W6.0_SMNR6045; symbol CBC_PCB:ZEMS0850-330M -> EasyEDA_Lib_2:SMNR6045-330MT; LCSC Part Name 33UH ±20% 6A 一体成型电感，合金电感，大电流，低阻抗 -> 33uH ±20% 1.65A; Manufacturer ZE(增益) -> SXN(顺翔诺); Manufacturer Part ZEMS0850-330M -> SMNR6045-330MT; Supplier Part C41438711 -> C135306
- Q601: renamed from Q8; footprint EasyEDA_Lib:TOLL-8_L10.4-W9.9-P1.20-LS11.7-BL -> CBC_PCB:DFN-8_L5.9-W5.2-P1.27-LS6.2-BL; symbol CBC_PCB:SP015N03BGHTO -> CBC_PCB:BSC320N20NS3G; LCSC Part Name 耐压:150V 电流:260A -> 1个N沟道 耐压:200V 电流:36A; Manufacturer Siliup(矽普) -> Infineon(英飞凌); Manufacturer Part SP015N03BGHTO -> BSC320N20NS3G; Supplier Part C22385354 -> C501501
- Q602: renamed from Q9; footprint EasyEDA_Lib:TOLL-8_L10.4-W9.9-P1.20-LS11.7-BL -> CBC_PCB:DFN-8_L5.9-W5.2-P1.27-LS6.2-BL; symbol CBC_PCB:SP015N03BGHTO -> CBC_PCB:BSC047N08NS3G; LCSC Part Name 耐压:150V 电流:260A -> 1个N沟道 耐压:80V 电流:100A; Manufacturer Siliup(矽普) -> Infineon(英飞凌); Manufacturer Part SP015N03BGHTO -> BSC047N08NS3G; Supplier Part C22385354 -> C501500
- U603: renamed from C62; value 2.2uF -> 1uF; footprint EasyEDA_Lib:CAP-TH_BD5.0-P2.00-D0.5-FD-1 -> EasyEDA_Lib_2:C0805; symbol CBC_PCB:ERJ1KM2R2D11OT -> EasyEDA_Lib_2:CC0805KKX7R0BB105; LCSC Part Name 2.2uF ±20% 100V -> 1uF ±10% 100V; Manufacturer AISHI(艾华集团) -> YAGEO(国巨); Manufacturer Part ERJ1KM2R2D11OT -> CC0805KKX7R0BB105; Supplier Part C694099 -> C5370002
- renumbered C41 to C607, C95 to C608, C15 to C610, C7 to C611, C59 to C612, C60 to C614, C63 to C615, C35 to C616, C96 to C617, C74 to C618, C97 to C619, C38 to C620, C98 to C621, C40 to C622, C99 to C623, C61 to C624, C67 to C625, C43 to C626, C100 to C627, C68 to C628, C66 to C629, C69 to C630, C70 to C631, U29 to C632, C71 to C633, C45 to C634, C101 to C635, C46 to C636, C102 to C637, C72 to C638, C44 to C639, C103 to C640, C77 to C641, C42 to C642, C104 to C643, C73 to C645, D17 to D603, D18 to D604, D16 to D605, D15 to D606, D29 to D607, D19 to D608, D21 to D609, D20 to D610, F4 to F601, F5 to F602, F6 to F603, L5 to L604, LED5 to LED601, LED6 to LED602, LED7 to LED603, R40 to R601, R43 to R602, R42 to R603, R31 to R604, R30 to R605, R58 to R606, R59 to R607, R37 to R608, R38 to R609, R39 to R610, R36 to R611, R6 to R612, R32 to R613, R33 to R614, R60 to R615, R61 to R616, R41 to R617, R5 to R618, R17 to R619, R66 to R620, R18 to R621, R67 to R622, R45 to R623, R44 to R624, R68 to R625, R19 to R626, R62 to R627, U23 to U601, U35 to U602, U8 to U604, U9 to U605, U27 to U606, U15 to U607, U37 to U608, U30 to U609, U28 to U610, U24 to U611, U36 to U612, U38 to U613, U39 to U614
Connections:
- net GND: now also C601.1, C602.1, C603.1, C604.1, C609.2, C613.2, C605.2, C606.2; no longer C601.2, C602.2, C603.2, C604.2, C609.1, C613.1, D601.2 (A), D602.2 (A)
- net GNDE: now also C644.1, C646.1, Q602.1 (S); no longer C644.2, C646.2, Q602.2 (S), Q602.3 (S), Q602.4 (S), Q602.5 (S), Q602.6 (S), Q602.7 (S), Q602.8 (S)
- net H_PWR-IN: now also C601.2, C602.2, C603.2, C604.2, C609.1, C605.1, C606.1; no longer C601.1, C602.1, C603.1, C604.1, C609.2
- net at Q601.1 (S): now also R617.2, U606.2; no longer R611.2
- net at D604.2 (A), L604.1, L604.2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: now also Q601.3 (D); no longer Q601.9 (D)
- net at C607.1, L602.1, U601.5 (SW): now also D601.2 (K); no longer D601.3 (K)
- net at C633.2, C638.2, C641.2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: now also C644.2, C646.2; no longer C644.1, C646.1
- net at D608.2 (A), L604.7, L604.8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: now also Q602.3 (D); no longer Q602.9 (D)
- net at C608.1, L603.1, U602.5 (SW): now also D602.2 (K); no longer D602.3 (K)
- net at R603.1: now also C613.1; no longer C613.2
- net at U610.1 (GATE): now also Q602.2 (G); no longer Q602.1 (G)
- new net: Q601.2 (G), R611.2
Other:
- moved on the sheet: C613
