File: engineering/electronics/pcbs/CBC_PCB/kicad/ESP32 SECTION.kicad_sch (KiCad schematic)
At the start: 20 parts, among them U2 2.4GHz

Commit message: fix(cbc): integrate ordered PCB update
Parts:
- removed C21: 100nF, EasyEDA_Lib:C0402, symbol CBC_PCB:CC0402KRX7R7BB104
- USB301: renamed from USB1; footprint EasyEDA_Lib:USB-C-SMD_TYPE-C-16PIN-2MD-073 -> EasyEDA_Lib_2:USB-C-SMD_TYPEC-303-ACP16; symbol CBC_PCB:TYPE-C 16PIN 2MD(073) -> EasyEDA_Lib_2:TYPEC-303-ACP16; LCSC Part Name Type-C 母 卧贴 -> Type-C 母 立贴; Manufacturer SHOU HAN(首韩) -> XUNPU(讯普); Manufacturer Part TYPE-C 16PIN 2MD(073) -> TYPEC-303-ACP16; Supplier Part C2765186 -> C720628
- renumbered C18 to C301, C19 to C302, C1 to C303, C20 to C304, C22 to C305, C23 to C306, C24 to C307, D3 to D301, D4 to D302, LED1 to LED301, Q1 to Q301, R7 to R301, R69 to R302, R8 to R303, R9 to R304, SW1 to SW301, U2 to U301, U7 to U302
Connections:
- net GND: now also USB301.1 (GND), USB301.2 (GND), USB301.3 (GND), USB301.4 (GND), USB301.A1 (GND), USB301.A12 (GND), USB301.B1 (GND), USB301.B12 (GND); no longer USB301.A1B12 (GND), USB301.B1A12 (GND)
- net USBV: now also USB301.A4 (VBUS), USB301.A9 (VBUS), USB301.B4 (VBUS), USB301.B9 (VBUS); no longer USB301.A4B9 (VBUS), USB301.B4A9 (VBUS)
- net DP_P: now reaches D302.1, USB301.A6 (DP1), USB301.B6 (DP2)
- net DP_N: now reaches D302.3, USB301.A7 (DN1), USB301.B7 (DN2)
Other:
- moved on the sheet: R303, R304
