File: engineering/electronics/pcbs/CBC_PCB/kicad/ESP32 SECTION.kicad_sch (KiCad schematic)
At the start: 19 parts, among them U301 2.4GHz

Commit message: feat(cbc): integrate PT1.5 CBC PCB update for the US build
Julius's CPC_PCB_21_10_26_5 package (issue #58): precharge ground fix with the new H_PWR-OUT- net and NT201, precharge and HV bus sensing, BZ501 buzzer, aux input inrush limiting (RT601, R628/R629, F604), BOM-review part swaps, and JLC production outputs. The board STEP is zipped because the raw export is 127 MB, which is over GitHub's 100 MB file limit.
Parts:
- U303: renamed from USB301; footprint EasyEDA_Lib_2:USB-C-SMD_TYPEC-303-ACP16 -> CBC_PCB:USB-C-TH_HANBO_MC-118LD-H65; symbol EasyEDA_Lib_2:TYPEC-303-ACP16 -> CBC_PCB:MC-118LD-H65; LCSC Part Name Type-C 母 立贴 -> Type-C 母 直插; Manufacturer XUNPU(讯普) -> HANBO(汉博); Manufacturer Part TYPEC-303-ACP16 -> MC-118LD-H65; Supplier Part C720628 -> C6332304
Connections:
- net GND: now also U303.13 (EH); no longer U303.1 (GND), U303.2 (GND), U303.3 (GND), U303.4 (GND)
- net BUZZER: now reaches U301.31 (IO38)
- net HV_BUS_SENSE: now reaches U301.38 (IO2)
- net PRECHARGE_SENSE: now reaches U301.39 (IO1)
- net at U303.A5 (CC1): now also R304.2; no longer R303.2
- net at U303.B5 (CC2): now also R303.2; no longer R304.2
- no-connect marks 34 -> 31
Other:
- note added: "rev PT1.5: IO1 = PRECHARGE_SENSE (ADC1_CH0), IO2 = HV_BUS_SENSE (ADC1_CH1), IO38 = BUZZER. Keep IO35-37 free (octal PSRAM on N16R8)."
