File: engineering/electronics/pcbs/CBC_PCB/kicad/CAN SECTION.kicad_sch (KiCad schematic)
At the start: 44 parts, among them U403 TJA1049T/3J, U404 ADM3053BRWZ-REEL7, X401 16MHz, X402 16MHz

Commit message: feat(cbc): integrate PT1.5 CBC PCB update for the US build
Julius's CPC_PCB_21_10_26_5 package (issue #58): precharge ground fix with the new H_PWR-OUT- net and NT201, precharge and HV bus sensing, BZ501 buzzer, aux input inrush limiting (RT601, R628/R629, F604), BOM-review part swaps, and JLC production outputs. The board STEP is zipped because the raw export is 127 MB, which is over GitHub's 100 MB file limit.
Parts:
- C411, C415: Manufacturer (none) -> YAGEO; Manufacturer Part (none) -> CC0805KRX7R9BB104; Supplier (none) -> LCSC; Supplier Part (none) -> C49678
- D401, D403: Manufacturer (none) -> Littelfuse; Manufacturer Part (none) -> PESD0603-240; Supplier (none) -> LCSC; Supplier Part (none) -> C2929617
- D402: LCSC Part Name 双向ESD 24V截止 峰值脉冲电流：3A@8/20us -> PESD1CAN-UX-ES; Manufacturer Nexperia(安世) -> ElecSuper; Manufacturer Part PESD1CAN-UX -> PESD1CAN-UX-ES; Supplier Part C152727 -> C19170883
- R403: Manufacturer (none) -> UNI-ROYAL; Manufacturer Part (none) -> 0805W8F0000T5E; Supplier (none) -> LCSC; Supplier Part (none) -> C17477
- R404: Manufacturer (none) -> UNI-ROYAL; Manufacturer Part (none) -> 0805W8F1002T5E; Supplier (none) -> LCSC; Supplier Part (none) -> C17414
- R407: Manufacturer YAGEO(国巨) -> UNI-ROYAL; Manufacturer Part RC0402FR-070RL -> 0402WGF0000TCE; Supplier Part C106231 -> C17168
- U403: Manufacturer (none) -> ZHHXDZ; Manufacturer Part (none) -> TJA1049T/3J-HX; Supplier (none) -> LCSC; Supplier Part (none) -> C53326714
