File: engineering/electronics/pcbs/CMAIN_PCB/kicad/CMAIN_PCB.kicad_pcb (KiCad board)
At the start: 4 copper layers, 210.2 x 220 mm, 258 parts, among them IC1 TSYS01, J1 RPI_5_WITH_SSQ-120-01-F-D, J10 1778719, J11 M9N-G4-3100, J12 B04B-JWPF-SK-R, J13 B04B-JWPF-SK-R, J14 XT30PW-F, J15 SM04B-GHS-TB_LF__SN_, J16 1778719, J17 SM03B-GHS-TB(LF)(SN), J19 1778719, J2 1778719, J21 1778719, J23 B04B-JWPF-SK-R, J24 1778719, J25 B08B-JWPF-SK-R, J26 B08B-JWPF-SK-R, J27 B04B-JWPF-SK-R, J28 B08B-JWPF-SK-R, J29 B06B-JWPF-SK-R, J3 AXK6S00547YG, J30 B06B-JWPF-SK-R, J31 B06B-JWPF-SK-R, J32 B04B-JWPF-SK-R, J34 B08B-JWPF-SK-R, J35 SM04B-GHS-TB_LF__SN_, J36 SM05B-GHS-TB_LF__SN_, J37 B04B-JWPF-SK-R, J38 B04B-JWPF-SK-R, J39 B04B-JWPF-SK-R, J4 AXK6S00547YG, J40 B04B-JWPF-SK-R, J41 SM06B-GHS-TB_LF__SN_, J42 B08B-JWPF-SK-R, J43 B04B-JWPF-SK-R, J44 B08B-JWPF-SK-R, J45 B04B-JWPF-SK-R, J46 B04B-JWPF-SK-R, J47 GIGABLOX_NANO_SWITCH_REVA_MOD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, J48 B04B-JWPF-SK-R, J49 B04B-JWPF-SK-R, J5 SM04B-GHS-TB_LF__SN_, J50 1814935, J51 GIGABLOX_NANO_SWITCH_REVA_MOD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, J52 B04B-JWPF-SK-R, J53 B04B-JWPF-SK-R, J55 B04B-JWPF-SK-R, J56 B04B-JWPF-SK-R, J57 B04B-JWPF-SK-R, J6 1778719, J7 SM04B-GHS-TB_LF__SN_, J8 B04B-JWPF-SK-R, J9 SM04B-GHS-TB_LF__SN_, K1 CPC1019N, K10 CPC1019N, K2 CPC1019N, K4 CPC1019N, K5 CPC1019N, K6 CPC1019N, K7 CPC1019N, K8 CPC1019N, K9 CPC1019N, Q1 SIRA99DP-T1-GE3, Q2 SIRA99DP-T1-GE3, Q4 PSMN4R3-30BL,118, Q5 PSMN4R3-30BL,118, Q6 PSMN4R3-30BL,118, Q7 PSMN4R3-30BL,118, Q8 PSMN4R3-30BL,118, Q9 PSMN4R3-30BL,118, U1 TJA1049T/3J, U10 SMTSO25100CTJ, U11 SMTSO25100CTJ, U12 SMTSO25100CTJ, U13 SMTWEM245STR, U14 SMTWEM245STR, U15 SMTWEM245STR, U16 SMTWEM245STR, U17 SY8205FCC, U18 SY8205FCC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

Commit message: electronics: shorten CMAIN footprint filenames for Windows
Parts:
- C1, C2, C25, C26, C27, C28, C29, C3, C30, C31, C32, C33, C35, C36, C37, C4, C40, C42, C43, C44, C5, C8: footprint CMAIN_PCB:C_0805_2012Metric_Pad1.18x1.45mm_HandSolder -> CMAIN_PCB:fp_71505040a9
- C22, C6, C7: footprint CMAIN_PCB:C_0603_1608Metric_Pad1.08x0.95mm_HandSolder -> CMAIN_PCB:fp_6a12138141
- J47, J51: footprint Snapeda:GIGABLOX_NANO_SWITCH_REVA_MODULE_LSHM-120-02.5-L-DV-A-S-K-TR -> Snapeda:fp_072ec239da
- JP1: footprint CMAIN_PCB:SolderJumper-2_P1.3mm_Bridged2Bar_RoundedPad1.0x1.5mm -> CMAIN_PCB:fp_fbc818f6a0
- JP2, JP5: footprint CMAIN_PCB:SolderJumper-2_P1.3mm_Open_RoundedPad1.0x1.5mm -> CMAIN_PCB:fp_e0a4172b1a
- Q1, Q2: footprint EasyEDA_Lib:POWERPAK-SO-8_L5.9-W4.9-P1.27-LS6.2-BL -> EasyEDA_Lib:fp_a2a0cc2e74
- R1, R10, R11, R12, R13, R14, R16, R17, R18, R19, R2, R20, R21, R22, R23, R24, R25, R26, R27, R28, R29, R3, R30, R31, R32, R33, R34, R35, R36, R37, R38, R39, R4, R40, R41, R42, R43, R44, R45, R46, R47, R48, R49, R5, R50, R51, R52, R53, R54, R55, R56, R57, R58, R59, R6, R7, R74, R75, R76, R77, R78, R79, R8, R9: footprint CMAIN_PCB:R_0805_2012Metric_Pad1.20x1.40mm_HandSolder -> CMAIN_PCB:fp_9fb50b8536
