File: engineering/electronics/pcbs/CMAIN_PCB/kicad/CMAIN_PCB.kicad_sch (KiCad schematic)
At the start: 72 parts, among them IC1 TSYS01, J1 RPI_5_WITH_SSQ-120-01-F-D, J10 1778719, J11 M9N-G4-3100, J12 1778719, J13 1778719, J14 XT30PW-F, J15 SM04B-GHS-TB_LF__SN_, J16 1778719, J17 SM03B-GHS-TB(LF)(SN), J18 SM04B-GHS-TB_LF__SN_, J19 1778719, J2 1778719, J20 SM04B-GHS-TB_LF__SN_, J21 1778719, J22 SM04B-GHS-TB_LF__SN_, J23 ${ALTIUM_VALUE}, J24 1778719, J27 ${ALTIUM_VALUE}, J29 1778735, J3 AXK6S00547YG, J30 1778735, J31 1814951, J32 ${ALTIUM_VALUE}, J33 USB4216-03-A, J35 SM04B-GHS-TB_LF__SN_, J36 SM05B-GHS-TB_LF__SN_, J37 1778719, J38 1778719, J39 1814935, J4 AXK6S00547YG, J40 ${ALTIUM_VALUE}, J41 SM06B-GHS-TB_LF__SN_, J45 ${ALTIUM_VALUE}, J49 1814935, J5 SM04B-GHS-TB_LF__SN_, J50 1814935, J53 1814935, J54 SM04B-GHS-TB_LF__SN_, J55 ${ALTIUM_VALUE}, J6 1778719, J7 SM04B-GHS-TB_LF__SN_, J8 1814935, J9 SM04B-GHS-TB_LF__SN_, U10 SMTSO25100CTJ, U11 SMTSO25100CTJ, U12 SMTSO25100CTJ, U3 SMTSOM380BTR, U5 C7429635, U6 SMTSOM380BTR, U7 SMTSOM380BTR, U8 SMTSOM380BTR, U9 SMTSO25100CTJ

Commit message: feat: integrate June PCB updates
Parts:
- removed TP1, TP2, TP3, TP4: TestPoint_Small, TestPoint:TestPoint_Pad_1.0x1.0mm, symbol Connector:TestPoint_Small
- J23, J27, J32, J40: value ${ALTIUM_VALUE} -> B04B-JWPF-SK-R; footprint CMAIN_PCB:1814948 -> CMAIN_PCB:B04B-JWPF-SK-R; symbol CMAIN_PCB:AT13-4P -> CMAIN_PCB:B04B-JWPF-SK-R; MFR Amphenol SINE Systems -> (none); MPN AT13-4P -> (none)
- J45, J55: value ${ALTIUM_VALUE} -> B04B-JWPF-SK-R; footprint CMAIN_PCB:AT13-4P -> CMAIN_PCB:B04B-JWPF-SK-R; symbol CMAIN_PCB:AT13-4P -> CMAIN_PCB:B04B-JWPF-SK-R; MFR Amphenol SINE Systems -> (none); MPN AT13-4P -> (none)
Connections:
- net CAN2_H: now also R14.1, S2.1 (NC_1)
- net  I2C2_SDA_GPS2_MAG_LED: no longer names the net of J3.83
- net BAT1_I: no longer names the net of J4.20
- net BAT1_V: no longer names the net of J4.18
- net BAT2_I: no longer names the net of J4.16
- net BAT2_V: no longer names the net of J4.14
- net I2C2_SCL: no longer names the net of J3.61
- net I2C2_SCL_GPS2_MAG_LED: no longer names the net of J3.85
- net I2C2_SDA: no longer names the net of J3.59
- net IO_RSSI_IN_AND_SBUS_OUT: no longer names the net of J4.57
- net SPEKTRUM_DSM_IN: no longer names the net of J4.59
- net UART7_CTS_TEL1: no longer names the net of J3.23
- net UART7_RTS_TEL1: no longer names the net of J3.21
- net VDD_3V3_SPEKTRUM: no longer names the net of J4.61
- net VDD_5V_GPS1: no longer names the net of J3.63
- net VDD_5V_GPS2: no longer names the net of J3.81
- net VDD_5V_I2C: no longer names the net of J3.57
- net VDD_5V_PPM_SBUS: no longer names the net of J4.53
- net VDD_5V_TEL1: no longer names the net of J3.19
- no-connect marks 183 -> 189
Other:
- note added: "BAT1_I"
- note added: "BAT1_V"
- note added: "BAT2_I"
- note added: "BAT2_V"
- note added: "I2C Temperature sensor for main PCB"
- note added: "I2C2_SCL"
- note added: "I2C2_SCL_GPS2_MAG_LED"
- note added: "I2C2_SDA"
- note added: "I2C2_SDA_GPS2_MAG_LED"
- note added: "IO_CH1 (PWM 1) IO_CH2 (PWM 2) IO_CH3 (PWM 3) IO_CH4 (PWM 4) IO_CH5 (PWM 5) IO_CH6 (PWM 6)"
- note added: "IO_CH5 (PWM6)"
- note added: "IO_RSSI_IN_AND_SBUS_OUT"
- note added: "Motor/ESC Connectors (Hobbywing X15)"
- note added: "Old Payload connectors"
- note added: "RPI header"
- note added: "Radar connectors"
- note added: "SIYI connectors"
- note added: "SPEKTRUM_DSM_IN"
- note added: "Threaded standoffs"
- note added: "Threaded standoffs for mounting the RPI"
- note added: "UART7_CTS_TEL1"
- note added: "UART7_RTS_TEL1"
- note added: "VDD_3V3_SPEKTRUM"
- note added: "VDD_5V_GPS1"
- note added: "VDD_5V_GPS2"
- note added: "VDD_5V_I2C"
- note added: "VDD_5V_PPM_SBUS"
- note added: "VDD_5V_TEL1"
- note removed: "IO_CH1 (PWM 1) IO_CH2 (PWM 2) IO_CH3 (PWM 3) IO_CH4 (PWM 4)"
- note removed: "Motor Connectors"
- note removed: "RPI (CAN+SIYI camera over ethernet)"
- note removed: "Radar connector"
- note removed: "Temp BC_PCB Temp BC_PCB"
- note removed: "Temperature sensor for main PCB"
- note removed: "mLRS RX"
- moved on the sheet: C1, IC1, J1, J10, J11, J12, J13, J14, J15, J16, J17, J18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

Commit message: electronics: update CMAIN PCB from June layout
Parts:
- added D5: (no value), EasyEDA_Lib_CMAIN:SOT-23-6_L2.9-W1.6-P0.95-LS2.8-BL, symbol EasyEDA_Lib_CMAIN:USBLC6-2SC6
- added D8: (no value), EasyEDA_Lib_CMAIN:SMA_L4.3-W2.6-LS5.0-FD, symbol EasyEDA_Lib_CMAIN:SS14_C7420316
- added J43, J46, J48, J52, J56: B04B-JWPF-SK-R, CMAIN_PCB:B04B-JWPF-SK-R, symbol CMAIN_PCB:B04B-JWPF-SK-R
- added U19, U20, U21, U5: (no value), EasyEDA_Lib_CMAIN:SMD_SMTSO3060CTJ, symbol EasyEDA_Lib_CMAIN:SMTSO3050CTJ
- CN18: renamed from J18; value SM04B-GHS-TB_LF__SN_ -> (none); footprint CMAIN_PCB:SM04B-GHS-TB -> EasyEDA_Lib_CMAIN:CONN-SMD_4P-P1.25_BM04B-GHS-TBT-LF-SN; symbol Samacsys:SM04B-GHS-TB_LF__SN_ -> EasyEDA_Lib_CMAIN:BM04B-GHS-TBT(LF)(SN); Height 5.1 -> (none); LCSC Part Name (none) -> 1x4P 间距:1.25mm 立贴 系列:GH; Manufacturer (none) -> JST; Manufacturer Part (none) -> BM04B-GHS-TBT(LF)(SN); Manufacturer_Name JST (JAPAN SOLDERLESS TERMINALS) -> (none); Manufacturer_Part_Number SM04B-GHS-TB(LF)(SN) -> (none); Mouser Part Number N/A -> (none); Mouser Price/Stock https://www.mouser.co.uk/ProductDetail/JST-Commercial/SM04B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 -> (none); Supplier (none) -> LCSC; Supplier Part (none) -> C161692
- CN20: renamed from J20; value SM04B-GHS-TB_LF__SN_ -> (none); footprint CMAIN_PCB:SM04B-GHS-TB -> EasyEDA_Lib_CMAIN:CONN-SMD_4P-P1.25_BM04B-GHS-TBT-LF-SN; symbol Samacsys:SM04B-GHS-TB_LF__SN_ -> EasyEDA_Lib_CMAIN:BM04B-GHS-TBT(LF)(SN); Height 5.1 -> (none); LCSC Part Name (none) -> 1x4P 间距:1.25mm 立贴 系列:GH; Manufacturer (none) -> JST; Manufacturer Part (none) -> BM04B-GHS-TBT(LF)(SN); Manufacturer_Name JST (JAPAN SOLDERLESS TERMINALS) -> (none); Manufacturer_Part_Number SM04B-GHS-TB(LF)(SN) -> (none); Mouser Part Number N/A -> (none); Mouser Price/Stock https://www.mouser.co.uk/ProductDetail/JST-Commercial/SM04B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 -> (none); Supplier (none) -> LCSC; Supplier Part (none) -> C161692
- CN22: renamed from J22; value SM04B-GHS-TB_LF__SN_ -> (none); footprint CMAIN_PCB:SM04B-GHS-TB -> EasyEDA_Lib_CMAIN:CONN-SMD_4P-P1.25_BM04B-GHS-TBT-LF-SN; symbol Samacsys:SM04B-GHS-TB_LF__SN_ -> EasyEDA_Lib_CMAIN:BM04B-GHS-TBT(LF)(SN); Height 5.1 -> (none); LCSC Part Name (none) -> 1x4P 间距:1.25mm 立贴 系列:GH; Manufacturer (none) -> JST; Manufacturer Part (none) -> BM04B-GHS-TBT(LF)(SN); Manufacturer_Name JST (JAPAN SOLDERLESS TERMINALS) -> (none); Manufacturer_Part_Number SM04B-GHS-TB(LF)(SN) -> (none); Mouser Part Number N/A -> (none); Mouser Price/Stock https://www.mouser.co.uk/ProductDetail/JST-Commercial/SM04B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 -> (none); Supplier (none) -> LCSC; Supplier Part (none) -> C161692
- CN54: renamed from J54; value SM04B-GHS-TB_LF__SN_ -> (none); footprint CMAIN_PCB:SM04B-GHS-TB -> EasyEDA_Lib_CMAIN:CONN-SMD_4P-P1.25_BM04B-GHS-TBT-LF-SN; symbol Samacsys:SM04B-GHS-TB_LF__SN_ -> EasyEDA_Lib_CMAIN:BM04B-GHS-TBT(LF)(SN); Height 5.1 -> (none); LCSC Part Name (none) -> 1x4P 间距:1.25mm 立贴 系列:GH; Manufacturer (none) -> JST; Manufacturer Part (none) -> BM04B-GHS-TBT(LF)(SN); Manufacturer_Name JST (JAPAN SOLDERLESS TERMINALS) -> (none); Manufacturer_Part_Number SM04B-GHS-TB(LF)(SN) -> (none); Mouser Part Number N/A -> (none); Mouser Price/Stock https://www.mouser.co.uk/ProductDetail/JST-Commercial/SM04B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 -> (none); Supplier (none) -> LCSC; Supplier Part (none) -> C161692
- J12, J13: value 1778719 -> B04B-JWPF-SK-R; footprint Samacsys:1778719 -> CMAIN_PCB:B04B-JWPF-SK-R; symbol Samacsys:1778719 -> CMAIN_PCB:B04B-JWPF-SK-R; Height 7.65 -> (none); Manufacturer_Name Phoenix Contact -> (none); Manufacturer_Part_Number 1778719 -> (none); Mouser Part Number 651-1778719 -> (none); Mouser Price/Stock https://www.mouser.co.uk/ProductDetail/Phoenix-Contact/1778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 -> (none)
- J29, J30: value 1778735 -> B06B-JWPF-SK-R; footprint CMAIN_PCB:1778735 -> CMAIN_PCB:B06B-JWPF-SK-R; symbol Samacsys_kicad_sym:1778735 -> CMAIN_PCB:B06B-JWPF-SK-R; Height 7.65 -> (none); Manufacturer_Name Phoenix Contact -> (none); Manufacturer_Part_Number 1778735 -> (none); Mouser Part Number 651-1778735 -> (none); Mouser Price/Stock https://www.mouser.co.uk/ProductDetail/Phoenix-Contact/1778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 -> (none)
- J31: value 1814951 -> B06B-JWPF-SK-R; footprint CMAIN_PCB:1814951 -> CMAIN_PCB:B06B-JWPF-SK-R; symbol Samacsys_kicad_sym:1814951 -> CMAIN_PCB:B06B-JWPF-SK-R; Height 5.1 -> (none); Manufacturer_Name Phoenix Contact -> (none); Manufacturer_Part_Number 1814951 -> (none); Mouser Part Number 651-1814951 -> (none); Mouser Price/Stock https://www.mouser.co.uk/ProductDetail/Phoenix-Contact/1814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 -> (none)
- J37, J38: value 1778719 -> B04B-JWPF-SK-R; footprint Samacsys:1778719 -> CMAIN_PCB:B04B-JWPF-SK-R; symbol Samacsys:1778719 -> CMAIN_PCB:B04B-JWPF-SK-R
- J39, J8: value 1814935 -> B04B-JWPF-SK-R; footprint CMAIN_PCB:1814935 -> CMAIN_PCB:B04B-JWPF-SK-R; symbol Samacsys_kicad_sym:1814935 -> CMAIN_PCB:B04B-JWPF-SK-R
- J49: value 1814935 -> B04B-JWPF-SK-R; footprint CMAIN_PCB:1814935 -> CMAIN_PCB:B04B-JWPF-SK-R; symbol Samacsys:1814935 -> CMAIN_PCB:B04B-JWPF-SK-R
- J53: value 1814935 -> B04B-JWPF-SK-R; footprint CMAIN_PCB:1814935 -> CMAIN_PCB:B04B-JWPF-SK-R; symbol Samacsys:1814935 -> CMAIN_PCB:B04B-JWPF-SK-R; Height 5.1 -> (none); Manufacturer_Name Phoenix Contact -> (none); Manufacturer_Part_Number 1814935 -> (none); Mouser Part Number 651-1814935 -> (none); Mouser Price/Stock https://www.mouser.co.uk/ProductDetail/Phoenix-Contact/1814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 -> (none)
- J57: renamed from U5; value C7429635 -> B04B-JWPF-SK-R; footprint CMAIN_PCB:CONN-TH_5P-P2.50_ZX-XH2.54-5PZZ -> CMAIN_PCB:B04B-JWPF-SK-R; symbol Snapeda:ZX-XH2.54-5PZZ -> CMAIN_PCB:B04B-JWPF-SK-R; Height 5.1 -> (none); LCSC Part Name 1x5P 间距:2.5mm 直插 系列:XH -> (none); Manufacturer Megastar(兆星) -> (none); Manufacturer Part ZX-XH2.54-5PZZ -> (none); Manufacturer_Name Phoenix Contact -> (none); Manufacturer_Part_Number 1814935 -> (none); Mouser Part Number 651-1814935 -> (none); Mouser Price/Stock https://www.mouser.co.uk/ProductDetail/Phoenix-Contact/1814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 -> (none); Supplier LCSC -> (none); Supplier Part C7429635 -> (none)
- USB33: renamed from J33; value USB4216-03-A -> (none); footprint CMAIN_PCB:USB421603A -> EasyEDA_Lib_CMAIN:USB-C-SMD_TYPEC-303-ACP16; symbol Samacsys_kicad_sym:USB4216-03-A -> EasyEDA_Lib_CMAIN:TYPEC-303-ACP16; Height 3.51 -> (none); LCSC Part Name (none) -> Type-C 母 立贴; Manufacturer (none) -> XUNPU(讯普); Manufacturer Part (none) -> TYPEC-303-ACP16; Manufacturer_Name GCT (GLOBAL CONNECTOR TECHNOLOGY) -> (none); Manufacturer_Part_Number USB4216-03-A -> (none); Mouser Part Number 640-USB4216-03-A -> (none); Mouser Price/Stock https://www.mouser.co.uk/ProductDetail/GCT/USB4216-03-A?qs=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 -> (none); Supplier (none) -> LCSC; Supplier Part (none) -> C720628
Connections:
- net 5V_1: now also CN18.1, CN22.1, J16.4, J19.4, J21.4, J24.4, J35.1, J4.67, J41.1, J9.1, D8.2 (K)
- net 5V_2: now also CN20.1, CN54.1, J1.2 (5V), J1.4 (5V), J5.1, J57.1, J6.3, J7.1
- net CAN1_H: now also J43.2, J46.2
- net CAN1_L: now also J43.3, J46.3
- net CAN2_H: now also J48.2, J56.2
- net CAN2_L: now also J48.3, J56.3
- net GND: now also R12.1, USB33.1 (GND), USB33.2 (GND), USB33.3 (GND), USB33.4 (GND), USB33.A12 (GND), USB33.B12 (GND), D5.2, J43.4, J46.4, J48.4, J52.3, J52.4, J56.4; no longer R12.2, USB33.G1 (GND_3), USB33.G2 (GND_4), USB33.G3 (GND_5), USB33.G4 (GND_6)
- net USB_D+: now also D5.6; no longer USB33.A6 (DP1)
- net USB_D-: now also D5.4; no longer USB33.A7 (DN1)
- net VBUS: now also USB33.A9 (VBUS), USB33.B9 (VBUS), D5.5, D8.1 (A)
- net at USB33.B5 (CC2): now also R13.2; no longer R12.1
- net at USB33.A5 (CC1): now also R12.2; no longer R13.2
- net at USB33.B6 (DP2): now also USB33.A6 (DP1), D5.1
- net at USB33.B7 (DN2): now also USB33.A7 (DN1), D5.3
- net +12V renamed 12V_1
- net 12V_1: no longer J49.4, J6.4, J8.4
- removed net +5V: CN18.1, CN20.1, CN22.1, CN54.1, J1.2 (5V), J1.4 (5V), J16.4, J19.4, J21.4, J24.4, J35.1, J4.67, J41.1, J5.1, J57.1, J6.3, J7.1, J9.1
- new net 12V_2: J49.4, J6.4, J8.4
- new net 12V_3: J52.1, J52.2
- new net 5V_3: J43.1, J46.1, J48.1, J56.1
- no-connect marks 189 -> 194
Other:
- added sheet Emergency_cutoff (Emergency_cutoff.kicad_sch)
- note added: "Emergency cutoff"
- note added: "New outside 12V connector"
- note added: "New outside CAN connectors"
- moved on the sheet: J21, J24, J35, J36, J41, J50, R12, R13

Commit message: electronics: shorten CMAIN footprint filenames for Windows
Parts:
- C1: footprint CMAIN_PCB:C_0805_2012Metric_Pad1.18x1.45mm_HandSolder -> CMAIN_PCB:fp_71505040a9
- JP1: footprint CMAIN_PCB:SolderJumper-2_P1.3mm_Bridged2Bar_RoundedPad1.0x1.5mm -> CMAIN_PCB:fp_fbc818f6a0
- JP2, JP5: footprint CMAIN_PCB:SolderJumper-2_P1.3mm_Open_RoundedPad1.0x1.5mm -> CMAIN_PCB:fp_e0a4172b1a
- R10, R11, R12, R13, R14, R2, R4, R5, R8: footprint CMAIN_PCB:R_0805_2012Metric_Pad1.20x1.40mm_HandSolder -> CMAIN_PCB:fp_9fb50b8536
Changed lines of the file:
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@@
 			)
 		)
-		(property "Footprint" "CMAIN_PCB:SolderJumper-2_P1.3mm_Bridged2Bar_RoundedPad1.0x1.5mm"
+		(property "Footprint" "CMAIN_PCB:fp_fbc818f6a0"
 			(at 434.34 129.286 0)
 			(hide yes)
@@
 			)
 		)
-		(property "Footprint" "CMAIN_PCB:C_0805_2012Metric_Pad1.18x1.45mm_HandSolder"
+		(property "Footprint" "CMAIN_PCB:fp_71505040a9"
 			(at 448.31 143.256 0)
 			(hide yes)
@@
 			)
 		)
-		(property "Footprint" "CMAIN_PCB:SolderJumper-2_P1.3mm_Open_RoundedPad1.0x1.5mm"
+		(property "Footprint" "CMAIN_PCB:fp_e0a4172b1a"
 			(at 450.85 166.116 0)
 			(hide yes)
@@
 			)
 		)
-		(property "Footprint" "CMAIN_PCB:R_0805_2012Metric_Pad1.20x1.40mm_HandSolder"
+		(property "Footprint" "CMAIN_PCB:fp_9fb50b8536"
 			(at 416.306 47.498 90)
 			(hide yes)
@@
 			)
 		)
-		(property "Footprint" "CMAIN_PCB:R_0805_2012Metric_Pad1.20x1.40mm_HandSolder"
+		(property "Footprint" "CMAIN_PCB:fp_9fb50b8536"
 			(at 430.53 169.926 90)
 			(hide yes)
@@
 			)
 		)
-		(property "Footprint" "CMAIN_PCB:R_0805_2012Metric_Pad1.20x1.40mm_HandSolder"
+		(property "Footprint" "CMAIN_PCB:fp_9fb50b8536"
 			(at 458.47 167.386 90)
 			(hide yes)
@@
 			)
 		)
-		(property "Footprint" "CMAIN_PCB:R_0805_2012Metric_Pad1.20x1.40mm_HandSolder"
+		(property "Footprint" "CMAIN_PCB:fp_9fb50b8536"
 			(at 446.532 345.694 0)
 			(hide yes)
@@
 			)
 		)
-		(property "Footprint" "CMAIN_PCB:SolderJumper-2_P1.3mm_Open_RoundedPad1.0x1.5mm"
+		(property "Footprint" "CMAIN_PCB:fp_e0a4172b1a"
 			(at 438.15 129.286 0)
 			(hide yes)
@@
 			)
 		)
-		(property "Footprint" "CMAIN_PCB:R_0805_2012Metric_Pad1.20x1.40mm_HandSolder"
+		(property "Footprint" "CMAIN_PCB:fp_9fb50b8536"
 			(at 456.438 340.868 0)
 			(hide yes)
@@
 			)
 		)
-		(property "Footprint" "CMAIN_PCB:R_0805_2012Metric_Pad1.20x1.40mm_HandSolder"
+		(property "Footprint" "CMAIN_PCB:fp_9fb50b8536"
 			(at 431.8 172.466 90)
 			(hide yes)
@@
 			)
 		)
-		(property "Footprint" "CMAIN_PCB:R_0805_2012Metric_Pad1.20x1.40mm_HandSolder"
+		(property "Footprint" "CMAIN_PCB:fp_9fb50b8536"
 			(at 435.61 136.906 90)
 			(hide yes)
@@
 			)
 		)
-		(property "Footprint" "CMAIN_PCB:R_0805_2012Metric_Pad1.20x1.40mm_HandSolder"
+		(property "Footprint" "CMAIN_PCB:fp_9fb50b8536"
 			(at 455.93 117.856 90)
 			(hide yes)
@@
 			)
 		)
-		(property "Footprint" "CMAIN_PCB:R_0805_2012Metric_Pad1.20x1.40mm_HandSolder"
+		(property "Footprint" "CMAIN_PCB:fp_9fb50b8536"
 			(at 439.42 136.906 90)
 			(hide yes)
