File: engineering/electronics/pcbs/CMAIN_PCB/kicad/power_supply.kicad_sch (KiCad schematic)
At the start: 108 parts, among them J25 ${ALTIUM_VALUE}, J26 ${ALTIUM_VALUE}, J28 ${ALTIUM_VALUE}, J34 ${ALTIUM_VALUE}, J42 ${ALTIUM_VALUE}, J44 ${ALTIUM_VALUE}, Q4 PSMN4R3-30BL,118, Q5 PSMN4R3-30BL,118, Q6 ${ALTIUM_VALUE}, Q7 ${ALTIUM_VALUE}, Q8 PSMN4R3-30BL,118, Q9 ${ALTIUM_VALUE}, U17 SY8205FCC, U18 SY8205FCC, U29 LTC4370IMS#PBF, U30 LTC4370IMS#PBF, U31 LTC4370IMS#PBF, U4 SY8205FCC

Commit message: feat: integrate June PCB updates
Parts:
- J25, J26, J28, J34, J42, J44: value ${ALTIUM_VALUE} -> B08B-JWPF-SK-R; footprint CMAIN_PCB:AT13-08PA-BM01 -> CMAIN_PCB:B08BJWPFSKRLFSN; symbol CMAIN_PCB:AT13-08PA-BM01 -> CMAIN_PCB:B08B-JWPF-SK-R; ALTIUM_VALUE AT13-08PA-BM01 -> (none); MFR Amphenol SINE Systems -> (none); MPN AT13-08PA-BM01 -> (none); SUPPLIER Mouser -> (none); SUPPLIER PART NUMBER 654-AT13-08PA-BM01 -> (none)

Commit message: electronics: update CMAIN PCB from June layout
Parts:
- C2, C25, C26, C33, C35, C36, C37, C40, C42, C43, C44, C8: footprint (none) -> CMAIN_PCB:C_0805_2012Metric_Pad1.18x1.45mm_HandSolder
- C22: footprint (none) -> CMAIN_PCB:C_0603_1608Metric_Pad1.08x0.95mm_HandSolder
- C38, C45: footprint (none) -> CMAIN_PCB:C_0603_1608Metric
- J25, J26, J28, J34, J42, J44: footprint CMAIN_PCB:B08BJWPFSKRLFSN -> CMAIN_PCB:B08B-JWPF-SK-R
- L1, L2, L3: value 4.7uH to 10uH (Saturation Current higher 6A, low DCR) -> 3.3uH; footprint (none) -> EasyEDA_Lib_CMAIN:IND-SMD_CYA0650-3.3UH; symbol Device:L -> EasyEDA_Lib_CMAIN:CYA0650-3.3UH; LCSC Part Name (none) -> 3.3uH ±20%; Manufacturer (none) -> SHOU HAN(首韩); Manufacturer Part (none) -> CYA0650-3.3UH; Supplier (none) -> LCSC; Supplier Part (none) -> C5189753
- R23, R24, R25, R34, R35, R36, R37, R38: footprint (none) -> CMAIN_PCB:R_0805_2012Metric_Pad1.20x1.40mm_HandSolder
Connections:
- net 12V_1: no longer C33.1, C34.1, C40.1, C41.1, R33.1, R36.1, R69.2, R70.2, R71.2, R72.2, R75.2, R76.2, U17.7 (PVIN), U17.8 (PVIN), U18.7 (PVIN), U18.8 (PVIN)
- net GND: now also D12.2 (A), D13.2 (A), D14.2 (A), D15.2 (A), D16.2 (A), D17.2 (A), LED1.1 (C), LED10.1 (C), LED11.1 (C), LED12.1 (C), LED13.1 (C), LED14.1 (C), LED15.1 (C), LED2.1 (C), LED3.1 (C), LED7.1 (C), LED8.1 (C), LED9.1 (C); no longer D12.A, D13.A, D14.A, D15.A, D16.A, D17.A, LED1.C, LED10.C, LED11.C, LED12.C, LED13.C, LED14.C, LED15.C, LED2.C, LED3.C, LED7.C, LED8.C, LED9.C
- net at Q7.1 (S): now also C12.2, C18.1, D15.1 (C), J34.3, J34.4, R53.2, U30.13 (VIN1); no longer U30.12 (GATE1)
- net at R70.1, U30.10 (OUT1): now also Q7.3 (D); no longer Q7.2 (D)
- net at R71.1, U31.7 (OUT2): now also Q8.3 (D); no longer Q8.2 (D)
- net at R67.1, U29.7 (OUT2): now also Q4.3 (D); no longer Q4.2 (D)
- net at C16.2, C21.1, J44.3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: now also D17.1 (C), Q9.1 (S); no longer D17.C, Q9.3 (S)
- net at Q5.1 (S): now also C11.2, C14.1, D14.1 (C), J28.3, J28.4, R52.2, U30.4 (VIN2); no longer U30.5 (GATE2)
- net at R69.1, U30.7 (OUT2): now also Q5.3 (D); no longer Q5.2 (D)
- net at R76.1: now also LED12.2 (A); no longer LED12.A
- net at R54.1: now also LED10.2 (A); no longer LED10.A
- net at C15.2, C20.1, J42.3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: now also D16.1 (C), Q8.1 (S); no longer D16.C, Q8.3 (S)
- net at R52.1: now also LED3.2 (A); no longer LED3.A
- net at R72.1, U31.10 (OUT1): now also Q9.3 (D); no longer Q9.2 (D)
- net at C10.2, C17.1, J26.3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: now also D13.1 (C), Q6.1 (S); no longer D13.C, Q6.3 (S)
- net at R51.1: now also LED8.2 (A); no longer LED8.A
- net at Q4.1 (S): now also C13.1, C9.2, D12.1 (C), J25.3, J25.4, R50.2, U29.4 (VIN2); no longer U29.5 (GATE2)
- net at U31.12 (GATE1): now also Q9.2 (G); no longer Q9.1 (G)
- net at R55.1: now also LED11.2 (A); no longer LED11.A
- net at R78.1: now also LED14.2 (A); no longer LED14.A
- net at R79.1: now also LED15.2 (A); no longer LED15.A
- net at U29.12 (GATE1): now also Q6.2 (G); no longer Q6.1 (G)
- net at R68.1, U29.10 (OUT1): now also Q6.3 (D); no longer Q6.2 (D)
- net at R77.1: now also LED13.2 (A); no longer LED13.A
- net at R53.1: now also LED9.2 (A); no longer LED9.A
- net at R75.1: now also LED7.2 (A); no longer LED7.A
- net at R50.1: now also LED1.2 (A); no longer LED1.A
- net at U31.5 (GATE2): now also Q8.2 (G); no longer Q8.1 (G)
- net at R74.1: now also LED2.2 (A); no longer LED2.A
- net GND_TR_1 renamed 12V_TR_SUPPLY_1
- net GND_TR_2 renamed 12V_TR_SUPPLY_2
- net GND_TR_3 renamed 12V_TR_SUPPLY_3
- net GND_TR_4 renamed 12V_TR_SUPPLY_4
- net GND_TR_5 renamed 12V_TR_SUPPLY_5
- net GND_TR_6 renamed 12V_TR_SUPPLY_6
- new net: Q7.2 (G), U30.12 (GATE1)
- new net: Q5.2 (G), U30.5 (GATE2)
- new net: Q4.2 (G), U29.5 (GATE2)
- new net 12V_2: C33.1, C34.1, R33.1, R69.2, R70.2, R75.2, U17.7 (PVIN), U17.8 (PVIN)
- new net 12V_3: C40.1, C41.1, R36.1, R71.2, R72.2, R76.2, U18.7 (PVIN), U18.8 (PVIN)

Commit message: electronics: shorten CMAIN footprint filenames for Windows
Parts:
- C2, C25, C26, C27, C28, C29, C30, C31, C32, C33, C35, C36, C37, C40, C42, C43, C44, C8: footprint CMAIN_PCB:C_0805_2012Metric_Pad1.18x1.45mm_HandSolder -> CMAIN_PCB:fp_71505040a9
- C22: footprint CMAIN_PCB:C_0603_1608Metric_Pad1.08x0.95mm_HandSolder -> CMAIN_PCB:fp_6a12138141
- R23, R24, R25, R33, R34, R35, R36, R37, R38, R50, R51, R52, R53, R54, R55, R74, R75, R76, R77, R78, R79: footprint CMAIN_PCB:R_0805_2012Metric_Pad1.20x1.40mm_HandSolder -> CMAIN_PCB:fp_9fb50b8536
Changed lines of the file:
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@@
 			)
 		)
-		(property "Footprint" "CMAIN_PCB:R_0805_2012Metric_Pad1.20x1.40mm_HandSolder"
+		(property "Footprint" "CMAIN_PCB:fp_9fb50b8536"
 			(at 402.59 203.2 0)
 			(hide yes)
@@
 			)
 		)
-		(property "Footprint" "CMAIN_PCB:C_0805_2012Metric_Pad1.18x1.45mm_HandSolder"
+		(property "Footprint" "CMAIN_PCB:fp_71505040a9"
 			(at 373.38 281.94 0)
 			(hide yes)
@@
 			)
 		)
-		(property "Footprint" "CMAIN_PCB:C_0805_2012Metric_Pad1.18x1.45mm_HandSolder"
+		(property "Footprint" "CMAIN_PCB:fp_71505040a9"
 			(at 340.36 200.66 0)
 			(hide yes)
@@
 			)
 		)
-		(property "Footprint" "CMAIN_PCB:R_0805_2012Metric_Pad1.20x1.40mm_HandSolder"
+		(property "Footprint" "CMAIN_PCB:fp_9fb50b8536"
 			(at 191.77 278.13 0)
 			(hide yes)
@@
 			)
 		)
-		(property "Footprint" "CMAIN_PCB:C_0805_2012Metric_Pad1.18x1.45mm_HandSolder"
+		(property "Footprint" "CMAIN_PCB:fp_71505040a9"
 			(at 205.74 203.2 0)
 			(hide yes)
@@
 			)
 		)
-		(property "Footprint" "CMAIN_PCB:R_0805_2012Metric_Pad1.20x1.40mm_HandSolder"
+		(property "Footprint" "CMAIN_PCB:fp_9fb50b8536"
 			(at 191.77 130.81 0)
 			(hide yes)
@@
 			)
 		)
-		(property "Footprint" "CMAIN_PCB:C_0805_2012Metric_Pad1.18x1.45mm_HandSolder"
+		(property "Footprint" "CMAIN_PCB:fp_71505040a9"
 			(at 212.09 281.94 0)
 			(hide yes)
@@
 			)
 		)
-		(property "Footprint" "CMAIN_PCB:C_0805_2012Metric_Pad1.18x1.45mm_HandSolder"
+		(property "Footprint" "CMAIN_PCB:fp_71505040a9"
 			(at 205.74 109.22 0)
 			(hide yes)
@@
 			)
 		)
-		(property "Footprint" "CMAIN_PCB:R_0805_2012Metric_Pad1.20x1.40mm_HandSolder"
+		(property "Footprint" "CMAIN_PCB:fp_9fb50b8536"
 			(at 337.82 99.06 0)
 			(hide yes)
@@
 			)
 		)
-		(property "Footprint" "CMAIN_PCB:C_0805_2012Metric_Pad1.18x1.45mm_HandSolder"
+		(property "Footprint" "CMAIN_PCB:fp_71505040a9"
 			(at 322.58 88.9 0)
 			(hide yes)
@@
 			)
 		)
-		(property "Footprint" "CMAIN_PCB:R_0805_2012Metric_Pad1.20x1.40mm_HandSolder"
+		(property "Footprint" "CMAIN_PCB:fp_9fb50b8536"
 			(at 402.59 195.58 0)
 			(hide yes)
@@
 			)
 		)
-		(property "Footprint" "CMAIN_PCB:R_0805_2012Metric_Pad1.20x1.40mm_HandSolder"
+		(property "Footprint" "CMAIN_PCB:fp_9fb50b8536"
 			(at 279.4 280.67 0)
 			(hide yes)
@@
 			)
 		)
-		(property "Footprint" "CMAIN_PCB:R_0805_2012Metric_Pad1.20x1.40mm_HandSolder"
+		(property "Footprint" "CMAIN_PCB:fp_9fb50b8536"
 			(at 191.77 325.12 0)
 			(hide yes)
@@
 			)
 		)
-		(property "Footprint" "CMAIN_PCB:C_0805_2012Metric_Pad1.18x1.45mm_HandSolder"
+		(property "Footprint" "CMAIN_PCB:fp_71505040a9"
 			(at 340.36 106.68 0)
 			(hide yes)
@@
 			)
 		)
-		(property "Footprint" "CMAIN_PCB:C_0805_2012Metric_Pad1.18x1.45mm_HandSolder"
+		(property "Footprint" "CMAIN_PCB:fp_71505040a9"
 			(at 212.09 181.61 0)
 			(hide yes)
@@
 			)
 		)
-		(property "Footprint" "CMAIN_PCB:R_0805_2012Metric_Pad1.20x1.40mm_HandSolder"
+		(property "Footprint" "CMAIN_PCB:fp_9fb50b8536"
 			(at 441.96 104.14 0)
 			(hide yes)
@@
 			)
 		)
-		(property "Footprint" "CMAIN_PCB:R_0805_2012Metric_Pad1.20x1.40mm_HandSolder"
+		(property "Footprint" "CMAIN_PCB:fp_9fb50b8536"
 			(at 401.32 295.91 0)
 			(hide yes)
@@
 			)
 		)
-		(property "Footprint" "CMAIN_PCB:R_0805_2012Metric_Pad1.20x1.40mm_HandSolder"
+		(property "Footprint" "CMAIN_PCB:fp_9fb50b8536"
 			(at 337.82 193.04 0)
 			(hide yes)
@@
 			)
 		)
-		(property "Footprint" "CMAIN_PCB:C_0603_1608Metric_Pad1.08x0.95mm_HandSolder"
+		(property "Footprint" "CMAIN_PCB:fp_6a12138141"
 			(at 392.43 101.6 0)
 			(hide yes)
@@
 			)
 		)
-		(property "Footprint" "CMAIN_PCB:C_0805_2012Metric_Pad1.18x1.45mm_HandSolder"
+		(property "Footprint" "CMAIN_PCB:fp_71505040a9"
 			(at 373.38 101.6 0)
 			(hide yes)
@@
 			)
 		)
-		(property "Footprint" "CMAIN_PCB:R_0805_2012Metric_Pad1.20x1.40mm_HandSolder"
+		(property "Footprint" "CMAIN_PCB:fp_9fb50b8536"
 			(at 445.77 298.45 0)
 			(hide yes)
@@
 			)
 		)
-		(property "Footprint" "CMAIN_PCB:R_0805_2012Metric_Pad1.20x1.40mm_HandSolder"
+		(property "Footprint" "CMAIN_PCB:fp_9fb50b8536"
 			(at 191.77 224.79 0)
 			(hide yes)
@@
 			)
 		)
-		(property "Footprint" "CMAIN_PCB:R_0805_2012Metric_Pad1.20x1.40mm_HandSolder"
+		(property "Footprint" "CMAIN_PCB:fp_9fb50b8536"
 			(at 401.32 303.53 0)
 			(hide yes)
@@
 			)
 		)
-		(property "Footprint" "CMAIN_PCB:R_0805_2012Metric_Pad1.20x1.40mm_HandSolder"
+		(property "Footprint" "CMAIN_PCB:fp_9fb50b8536"
 			(at 279.4 180.34 0)
 			(hide yes)
@@
 			)
 		)
-		(property "Footprint" "CMAIN_PCB:C_0805_2012Metric_Pad1.18x1.45mm_HandSolder"
+		(property "Footprint" "CMAIN_PCB:fp_71505040a9"
 			(at 374.65 181.61 0)
 			(hide yes)
@@
 			)
 		)
-		(property "Footprint" "CMAIN_PCB:C_0805_2012Metric_Pad1.18x1.45mm_HandSolder"
+		(property "Footprint" "CMAIN_PCB:fp_71505040a9"
 			(at 212.09 87.63 0)
 			(hide yes)
@@
 			)
 		)
-		(property "Footprint" "CMAIN_PCB:R_0805_2012Metric_Pad1.20x1.40mm_HandSolder"
+		(property "Footprint" "CMAIN_PCB:fp_9fb50b8536"
 			(at 438.15 198.12 0)
 			(hide yes)
@@
 			)
 		)
-		(property "Footprint" "CMAIN_PCB:C_0805_2012Metric_Pad1.18x1.45mm_HandSolder"
+		(property "Footprint" "CMAIN_PCB:fp_71505040a9"
 			(at 322.58 182.88 0)
 			(hide yes)
@@
 			)
 		)
-		(property "Footprint" "CMAIN_PCB:R_0805_2012Metric_Pad1.20x1.40mm_HandSolder"
+		(property "Footprint" "CMAIN_PCB:fp_9fb50b8536"
 			(at 336.55 293.37 0)
 			(hide yes)
@@
 			)
 		)
-		(property "Footprint" "CMAIN_PCB:R_0805_2012Metric_Pad1.20x1.40mm_HandSolder"
+		(property "Footprint" "CMAIN_PCB:fp_9fb50b8536"
 			(at 402.59 109.22 0)
 			(hide yes)
@@
 			)
 		)
-		(property "Footprint" "CMAIN_PCB:R_0805_2012Metric_Pad1.20x1.40mm_HandSolder"
+		(property "Footprint" "CMAIN_PCB:fp_9fb50b8536"
 			(at 402.59 101.6 0)
 			(hide yes)
@@
 			)
 		)
-		(property "Footprint" "CMAIN_PCB:C_0805_2012Metric_Pad1.18x1.45mm_HandSolder"
+		(property "Footprint" "CMAIN_PCB:fp_71505040a9"
 			(at 321.31 283.21 0)
 			(hide yes)
@@
 			)
 		)
-		(property "Footprint" "CMAIN_PCB:C_0805_2012Metric_Pad1.18x1.45mm_HandSolder"
+		(property "Footprint" "CMAIN_PCB:fp_71505040a9"
 			(at 374.65 87.63 0)
 			(hide yes)
@@
 			)
 		)
-		(property "Footprint" "CMAIN_PCB:C_0805_2012Metric_Pad1.18x1.45mm_HandSolder"
+		(property "Footprint" "CMAIN_PCB:fp_71505040a9"
 			(at 205.74 303.53 0)
 			(hide yes)
@@
 			)
 		)
-		(property "Footprint" "CMAIN_PCB:C_0805_2012Metric_Pad1.18x1.45mm_HandSolder"
+		(property "Footprint" "CMAIN_PCB:fp_71505040a9"
 			(at 339.09 300.99 0)
 			(hide yes)
@@
 			)
 		)
-		(property "Footprint" "CMAIN_PCB:C_0805_2012Metric_Pad1.18x1.45mm_HandSolder"
+		(property "Footprint" "CMAIN_PCB:fp_71505040a9"
 			(at 372.11 295.91 0)
 			(hide yes)
@@
 			)
 		)
-		(property "Footprint" "CMAIN_PCB:R_0805_2012Metric_Pad1.20x1.40mm_HandSolder"
+		(property "Footprint" "CMAIN_PCB:fp_9fb50b8536"
 			(at 191.77 177.8 0)
 			(hide yes)
@@
 			)
 		)
-		(property "Footprint" "CMAIN_PCB:R_0805_2012Metric_Pad1.20x1.40mm_HandSolder"
+		(property "Footprint" "CMAIN_PCB:fp_9fb50b8536"
 			(at 191.77 83.82 0)
 			(hide yes)
@@
 			)
 		)
-		(property "Footprint" "CMAIN_PCB:R_0805_2012Metric_Pad1.20x1.40mm_HandSolder"
+		(property "Footprint" "CMAIN_PCB:fp_9fb50b8536"
 			(at 279.4 86.36 0)
 			(hide yes)
@@
 			)
 		)
-		(property "Footprint" "CMAIN_PCB:C_0805_2012Metric_Pad1.18x1.45mm_HandSolder"
+		(property "Footprint" "CMAIN_PCB:fp_71505040a9"
 			(at 373.38 195.58 0)
 			(hide yes)

Commit message: electronics: integrate CMAIN STEP updates and consolidate footprints
Parts:
- F2, F3, F4: footprint Samacsys:0154005DR -> CMAIN_PCB:0154005DR
- L1, L2, L3: footprint EasyEDA_Lib_CMAIN:IND-SMD_CYA0650-3.3UH -> EasyEDA_Lib:IND-SMD_CYA0650-3.3UH
Changed lines of the file:
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@@
 			)
 		)
-		(property "Footprint" "EasyEDA_Lib_CMAIN:IND-SMD_CYA0650-3.3UH"
+		(property "Footprint" "EasyEDA_Lib:IND-SMD_CYA0650-3.3UH"
 			(at 386.08 99.06 0)
 			(hide yes)
@@
 			)
 		)
-		(property "Footprint" "Samacsys:0154005DR"
+		(property "Footprint" "CMAIN_PCB:0154005DR"
 			(at 436.88 195.58 0)
 			(hide yes)
@@
 			)
 		)
-		(property "Footprint" "EasyEDA_Lib_CMAIN:IND-SMD_CYA0650-3.3UH"
+		(property "Footprint" "EasyEDA_Lib:IND-SMD_CYA0650-3.3UH"
 			(at 386.334 193.04 0)
 			(hide yes)
@@
 	(symbol
 		(lib_id "power:PWR_FLAG")
+		(at 369.57 284.48 0)
+		(unit 1)
+		(body_style 1)
+		(exclude_from_sim no)
+		(in_bom yes)
+		(on_board yes)
+		(in_pos_files yes)
+		(dnp no)
+		(fields_autoplaced yes)
+		(property "Reference" "#FLG907"
+			(at 369.57 283.21 0)
+			(hide yes)
+			(show_name no)
+			(do_not_autoplace no)
+			(effects
+				(font
+					(size 1.27 1.27)
+				)
+			)
+		)
+		(property "Value" "PWR_FLAG"
+			(at 369.57 279.4 0)
+			(hide yes)
+			(show_name no)
+			(do_not_autoplace no)
+			(effects
+				(font
+					(size 1.27 1.27)
+				)
+			)
+		)
+		(property "Footprint" ""
+			(at 369.57 284.48 0)
+			(hide yes)
+			(show_name no)
+			(do_not_autoplace no)
+			(effects
+				(font
+					(size 1.27 1.27)
+				)
+			)
+		)
+		(property "Datasheet" ""
+			(at 369.57 284.48 0)
+			(hide yes)
+			(show_name no)
+			(do_not_autoplace no)
+			(effects
+				(font
+					(size 1.27 1.27)
+				)
+			)
+		)
+		(property "Description" "Special symbol for telling ERC where power comes from"
+			(at 369.57 284.48 0)
+			(hide yes)
+			(show_name no)
+			(do_not_autoplace no)
+			(effects
+				(font
+					(size 1.27 1.27)
+				)
+			)
+		)
+		(pin "1"
+		)
+		(instances
+			(project "CMAIN_PCB"
+				(path "/ca31b60c-f1cb-4b97-95b8-376c0a181311/002c9034-3e37-4b7e-9bfc-c61c7c67d734"
+					(reference "#FLG907")
+					(unit 1)
+				)
+			)
+		)
+	)
+	(symbol
+		(lib_id "power:PWR_FLAG")
 		(at 116.84 227.33 0)
 		(unit 1)
@@
 			)
 		)
-		(property "Footprint" "Samacsys:0154005DR"
+		(property "Footprint" "CMAIN_PCB:0154005DR"
 			(at 434.34 289.56 0)
 			(hide yes)
@@
 			)
 		)
-		(property "Footprint" "EasyEDA_Lib_CMAIN:IND-SMD_CYA0650-3.3UH"
+		(property "Footprint" "EasyEDA_Lib:IND-SMD_CYA0650-3.3UH"
 			(at 384.556 293.37 0)
 			(hide yes)
@@
 	)
 	(symbol
+		(lib_id "power:PWR_FLAG")
+		(at 370.84 184.15 0)
+		(unit 1)
+		(body_style 1)
+		(exclude_from_sim no)
+		(in_bom yes)
+		(on_board yes)
+		(in_pos_files yes)
+		(dnp no)
+		(fields_autoplaced yes)
+		(property "Reference" "#FLG906"
+			(at 370.84 182.88 0)
+			(hide yes)
+			(show_name no)
+			(do_not_autoplace no)
+			(effects
+				(font
+					(size 1.27 1.27)
+				)
+			)
+		)
+		(property "Value" "PWR_FLAG"
+			(at 370.84 179.07 0)
+			(hide yes)
+			(show_name no)
+			(do_not_autoplace no)
+			(effects
+				(font
+					(size 1.27 1.27)
+				)
+			)
+		)
+		(property "Footprint" ""
+			(at 370.84 184.15 0)
+			(hide yes)
+			(show_name no)
+			(do_not_autoplace no)
+			(effects
+				(font
+					(size 1.27 1.27)
+				)
+			)
+		)
+		(property "Datasheet" ""
+			(at 370.84 184.15 0)
+			(hide yes)
+			(show_name no)
+			(do_not_autoplace no)
+			(effects
+				(font
+					(size 1.27 1.27)
+				)
+			)
+		)
+		(property "Description" "Special symbol for telling ERC where power comes from"
+			(at 370.84 184.15 0)
+			(hide yes)
+			(show_name no)
+			(do_not_autoplace no)
+			(effects
+				(font
+					(size 1.27 1.27)
+				)
+			)
+		)
+		(pin "1"
+		)
+		(instances
+			(project "CMAIN_PCB"
+				(path "/ca31b60c-f1cb-4b97-95b8-376c0a181311/002c9034-3e37-4b7e-9bfc-c61c7c67d734"
+					(reference "#FLG906")
+					(unit 1)
+				)
+			)
+		)
+	)
+	(symbol
 		(lib_id "Device:R_Small")
 		(at 402.59 109.22 180)
@@
 			)
 		)
-		(property "Footprint" "Samacsys:0154005DR"
+		(property "Footprint" "CMAIN_PCB:0154005DR"
 			(at 438.15 389.89 0)
 			(hide yes)
@@
 					(unit 1)
 				)
-			)
-		)
-	)
-	(symbol
-		(lib_id "power:PWR_FLAG")
-		(at 370.84 184.15 0)
-		(unit 1)
-		(body_style 1)
-		(exclude_from_sim no)
-		(in_bom yes)
-		(on_board yes)
-		(in_pos_files yes)
-		(dnp no)
-		(fields_autoplaced yes)
-		(property "Reference" "#FLG906"
-			(at 370.84 182.88 0)
-			(hide yes)
-			(show_name no)
-			(do_not_autoplace no)
-			(effects
-				(font
-					(size 1.27 1.27)
-				)
-			)
-		)
-		(property "Value" "PWR_FLAG"
-			(at 370.84 179.07 0)
-			(hide yes)
-			(show_name no)
-			(do_not_autoplace no)
-			(effects
-				(font
-					(size 1.27 1.27)
-				)
-			)
-		)
-		(property "Footprint" ""
-			(at 370.84 184.15 0)
-			(hide yes)
-			(show_name no)
-			(do_not_autoplace no)
-			(effects
-				(font
-					(size 1.27 1.27)
-				)
-			)
-		)
-		(property "Datasheet" ""
-			(at 370.84 184.15 0)
-			(hide yes)
-			(show_name no)
-			(do_not_autoplace no)
-			(effects
-				(font
-					(size 1.27 1.27)
-				)
-			)
-		)
-		(property "Description" "Special symbol for telling ERC where power comes from"
-			(at 370.84 184.15 0)
-			(hide yes)
-			(show_name no)
-			(do_not_autoplace no)
-			(effects
-				(font
-					(size 1.27 1.27)
-				)
-			)
-		)
-		(pin "1"
-		)
-		(instances
-			(project "CMAIN_PCB"
-				(path "/ca31b60c-f1cb-4b97-95b8-376c0a181311/002c9034-3e37-4b7e-9bfc-c61c7c67d734"
-					(reference "#FLG906")
-					(unit 1)
-				)
-			)
-		)
-	)
-	(symbol
-		(lib_id "power:PWR_FLAG")
-		(at 369.57 284.48 0)
-		(unit 1)
-		(body_style 1)
-		(exclude_from_sim no)
-		(in_bom yes)
-		(on_board yes)
-		(in_pos_files yes)
-		(dnp no)
-		(fields_autoplaced yes)
-		(property "Reference" "#FLG907"
-			(at 369.57 283.21 0)
-			(hide yes)
-			(show_name no)
-			(do_not_autoplace no)
-			(effects
-				(font
-					(size 1.27 1.27)
-				)
-			)
-		)
-		(property "Value" "PWR_FLAG"
-			(at 369.57 279.40 0)
-			(hide yes)
-			(show_name no)
-			(do_not_autoplace no)
-			(effects
-				(font
-					(size 1.27 1.27)
-				)
-			)
-		)
-		(property "Footprint" ""
-			(at 369.57 284.48 0)
-			(hide yes)
-			(show_name no)
-			(do_not_autoplace no)
-			(effects
-				(font
-					(size 1.27 1.27)
-				)
-			)
-		)
-		(property "Datasheet" ""
-			(at 369.57 284.48 0)
-			(hide yes)
-			(show_name no)
-			(do_not_autoplace no)
-			(effects
-				(font
-					(size 1.27 1.27)
-				)
-			)
-		)
-		(property "Description" "Special symbol for telling ERC where power comes from"
-			(at 369.57 284.48 0)
-			(hide yes)
-			(show_name no)
-			(do_not_autoplace no)
-			(effects
-				(font
-					(size 1.27 1.27)
-				)
-			)
-		)
-		(pin "1"
-		)
-		(instances
-			(project "CMAIN_PCB"
-				(path "/ca31b60c-f1cb-4b97-95b8-376c0a181311/002c9034-3e37-4b7e-9bfc-c61c7c67d734"
-					(reference "#FLG907")
-					(unit 1)
-				)

Commit message: Resolve CMAIN ERC warnings
Parts:
- L1, L2, L3: symbol EasyEDA_Lib_CMAIN:CYA0650-3.3UH -> CMAIN_PCB:CYA0650-3.3UH
Changed lines of the file:
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@@
 	)
 	(symbol
-		(lib_id "EasyEDA_Lib_CMAIN:CYA0650-3.3UH")
+		(lib_id "CMAIN_PCB:CYA0650-3.3UH")
 		(at 386.08 99.06 0)
 		(unit 1)
@@
 	)
 	(symbol
-		(lib_id "EasyEDA_Lib_CMAIN:CYA0650-3.3UH")
+		(lib_id "CMAIN_PCB:CYA0650-3.3UH")
 		(at 386.334 193.04 0)
 		(unit 1)
@@
 	)
 	(symbol
-		(lib_id "EasyEDA_Lib_CMAIN:CYA0650-3.3UH")
+		(lib_id "CMAIN_PCB:CYA0650-3.3UH")
 		(at 384.556 293.37 0)
 		(unit 1)
