File: engineering/electronics/pcbs/CMAIN_PCB/kicad/power_supply.kicad_sch (KiCad schematic)
At the start: 108 parts, among them J25 B08B-JWPF-SK-R, J26 B08B-JWPF-SK-R, J28 B08B-JWPF-SK-R, J34 B08B-JWPF-SK-R, J42 B08B-JWPF-SK-R, J44 B08B-JWPF-SK-R, Q4 PSMN4R3-30BL,118, Q5 PSMN4R3-30BL,118, Q6 PSMN4R3-30BL,118, Q7 PSMN4R3-30BL,118, Q8 PSMN4R3-30BL,118, Q9 PSMN4R3-30BL,118, U17 SY8205FCC, U18 SY8205FCC, U29 LTC4370IMS#PBF, U30 LTC4370IMS#PBF, U31 LTC4370IMS#PBF, U4 SY8205FCC

Commit message: fix(cmain): integrate prototype ordering update
Parts:
- D10: renamed from LED8; value RED -> APT2012SURCK; footprint CMAIN_PCB:LEDC2012X85N -> CMAIN_PCB:LED_APT2012SURCK; symbol Signal Distribution Box-altium-import:root_3_LED_SMD -> CMAIN_PCB:APT2012SURCK; ALTIUM_VALUE RED -> (none); Availability (none) -> In Stock; Check_prices (none) -> https://www.snapeda.com/parts/APT2012SURCK/Kingbright/view-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; MANUFACTURER (none) -> Kingbright; MAXIMUM_PACKAGE_HEIGHT (none) -> 0.75mm; MF (none) -> Kingbright; MFR ams OSRAM -> (none); MP (none) -> APT2012SURCK; MPN LS T676-Q1R2-1-Z -> (none); PARTREV (none) -> V.20B; PRICE 0.3 -> (none); Package (none) -> 0805 Kingbright; Price (none) -> None; STANDARD (none) -> Manufacturer Recommendations; SUPPLIER Mouser -> (none); SUPPLIER PART NUMBER 720-LST676-Q1R2-1-Z -> (none); SnapEDA_Link (none) -> https://www.snapeda.com/parts/APT2012SURCK/Kingbright/view-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
- D11: renamed from LED3; value RED -> APT2012SURCK; footprint CMAIN_PCB:LEDC2012X85N -> CMAIN_PCB:LED_APT2012SURCK; symbol Signal Distribution Box-altium-import:root_3_LED_SMD -> CMAIN_PCB:APT2012SURCK; ALTIUM_VALUE RED -> (none); Availability (none) -> In Stock; Check_prices (none) -> https://www.snapeda.com/parts/APT2012SURCK/Kingbright/view-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; MANUFACTURER (none) -> Kingbright; MAXIMUM_PACKAGE_HEIGHT (none) -> 0.75mm; MF (none) -> Kingbright; MFR ams OSRAM -> (none); MP (none) -> APT2012SURCK; MPN LS T676-Q1R2-1-Z -> (none); PARTREV (none) -> V.20B; PRICE 0.3 -> (none); Package (none) -> 0805 Kingbright; Price (none) -> None; STANDARD (none) -> Manufacturer Recommendations; SUPPLIER Mouser -> (none); SUPPLIER PART NUMBER 720-LST676-Q1R2-1-Z -> (none); SnapEDA_Link (none) -> https://www.snapeda.com/parts/APT2012SURCK/Kingbright/view-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
- D18: renamed from LED9; value RED -> APT2012SURCK; footprint CMAIN_PCB:LEDC2012X85N -> CMAIN_PCB:LED_APT2012SURCK; symbol Signal Distribution Box-altium-import:root_3_LED_SMD -> CMAIN_PCB:APT2012SURCK; ALTIUM_VALUE RED -> (none); Availability (none) -> In Stock; Check_prices (none) -> https://www.snapeda.com/parts/APT2012SURCK/Kingbright/view-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; MANUFACTURER (none) -> Kingbright; MAXIMUM_PACKAGE_HEIGHT (none) -> 0.75mm; MF (none) -> Kingbright; MFR ams OSRAM -> (none); MP (none) -> APT2012SURCK; MPN LS T676-Q1R2-1-Z -> (none); PARTREV (none) -> V.20B; PRICE 0.3 -> (none); Package (none) -> 0805 Kingbright; Price (none) -> None; STANDARD (none) -> Manufacturer Recommendations; SUPPLIER Mouser -> (none); SUPPLIER PART NUMBER 720-LST676-Q1R2-1-Z -> (none); SnapEDA_Link (none) -> https://www.snapeda.com/parts/APT2012SURCK/Kingbright/view-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
- D19: renamed from LED10; value RED -> APT2012SURCK; footprint CMAIN_PCB:LEDC2012X85N -> CMAIN_PCB:LED_APT2012SURCK; symbol Signal Distribution Box-altium-import:root_3_LED_SMD -> CMAIN_PCB:APT2012SURCK; ALTIUM_VALUE RED -> (none); Availability (none) -> In Stock; Check_prices (none) -> https://www.snapeda.com/parts/APT2012SURCK/Kingbright/view-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; MANUFACTURER (none) -> Kingbright; MAXIMUM_PACKAGE_HEIGHT (none) -> 0.75mm; MF (none) -> Kingbright; MFR ams OSRAM -> (none); MP (none) -> APT2012SURCK; MPN LS T676-Q1R2-1-Z -> (none); PARTREV (none) -> V.20B; PRICE 0.3 -> (none); Package (none) -> 0805 Kingbright; Price (none) -> None; STANDARD (none) -> Manufacturer Recommendations; SUPPLIER Mouser -> (none); SUPPLIER PART NUMBER 720-LST676-Q1R2-1-Z -> (none); SnapEDA_Link (none) -> https://www.snapeda.com/parts/APT2012SURCK/Kingbright/view-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
- D20: renamed from LED11; value RED -> APT2012SURCK; footprint CMAIN_PCB:LEDC2012X85N -> CMAIN_PCB:LED_APT2012SURCK; symbol Signal Distribution Box-altium-import:root_3_LED_SMD -> CMAIN_PCB:APT2012SURCK; ALTIUM_VALUE RED -> (none); Availability (none) -> In Stock; Check_prices (none) -> https://www.snapeda.com/parts/APT2012SURCK/Kingbright/view-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; MANUFACTURER (none) -> Kingbright; MAXIMUM_PACKAGE_HEIGHT (none) -> 0.75mm; MF (none) -> Kingbright; MFR ams OSRAM -> (none); MP (none) -> APT2012SURCK; MPN LS T676-Q1R2-1-Z -> (none); PARTREV (none) -> V.20B; PRICE 0.3 -> (none); Package (none) -> 0805 Kingbright; Price (none) -> None; STANDARD (none) -> Manufacturer Recommendations; SUPPLIER Mouser -> (none); SUPPLIER PART NUMBER 720-LST676-Q1R2-1-Z -> (none); SnapEDA_Link (none) -> https://www.snapeda.com/parts/APT2012SURCK/Kingbright/view-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
- D21: renamed from LED2; value RED -> APT2012SURCK; footprint CMAIN_PCB:LEDC2012X85N -> CMAIN_PCB:LED_APT2012SURCK; symbol Signal Distribution Box-altium-import:root_3_LED_SMD -> CMAIN_PCB:APT2012SURCK; ALTIUM_VALUE RED -> (none); Availability (none) -> In Stock; Check_prices (none) -> https://www.snapeda.com/parts/APT2012SURCK/Kingbright/view-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; MANUFACTURER (none) -> Kingbright; MAXIMUM_PACKAGE_HEIGHT (none) -> 0.75mm; MF (none) -> Kingbright; MFR ams OSRAM -> (none); MP (none) -> APT2012SURCK; MPN LS T676-Q1R2-1-Z -> (none); PARTREV (none) -> V.20B; PRICE 0.3 -> (none); Package (none) -> 0805 Kingbright; Price (none) -> None; STANDARD (none) -> Manufacturer Recommendations; SUPPLIER Mouser -> (none); SUPPLIER PART NUMBER 720-LST676-Q1R2-1-Z -> (none); SnapEDA_Link (none) -> https://www.snapeda.com/parts/APT2012SURCK/Kingbright/view-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
- D22: renamed from LED7; value RED -> APT2012SURCK; footprint CMAIN_PCB:LEDC2012X85N -> CMAIN_PCB:LED_APT2012SURCK; symbol Signal Distribution Box-altium-import:root_3_LED_SMD -> CMAIN_PCB:APT2012SURCK; ALTIUM_VALUE RED -> (none); Availability (none) -> In Stock; Check_prices (none) -> https://www.snapeda.com/parts/APT2012SURCK/Kingbright/view-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; MANUFACTURER (none) -> Kingbright; MAXIMUM_PACKAGE_HEIGHT (none) -> 0.75mm; MF (none) -> Kingbright; MFR ams OSRAM -> (none); MP (none) -> APT2012SURCK; MPN LS T676-Q1R2-1-Z -> (none); PARTREV (none) -> V.20B; PRICE 0.3 -> (none); Package (none) -> 0805 Kingbright; Price (none) -> None; STANDARD (none) -> Manufacturer Recommendations; SUPPLIER Mouser -> (none); SUPPLIER PART NUMBER 720-LST676-Q1R2-1-Z -> (none); SnapEDA_Link (none) -> https://www.snapeda.com/parts/APT2012SURCK/Kingbright/view-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
- D23: renamed from LED12; value RED -> APT2012SURCK; footprint CMAIN_PCB:LEDC2012X85N -> CMAIN_PCB:LED_APT2012SURCK; symbol Signal Distribution Box-altium-import:root_3_LED_SMD -> CMAIN_PCB:APT2012SURCK; ALTIUM_VALUE RED -> (none); Availability (none) -> In Stock; Check_prices (none) -> https://www.snapeda.com/parts/APT2012SURCK/Kingbright/view-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; MANUFACTURER (none) -> Kingbright; MAXIMUM_PACKAGE_HEIGHT (none) -> 0.75mm; MF (none) -> Kingbright; MFR ams OSRAM -> (none); MP (none) -> APT2012SURCK; MPN LS T676-Q1R2-1-Z -> (none); PARTREV (none) -> V.20B; PRICE 0.3 -> (none); Package (none) -> 0805 Kingbright; Price (none) -> None; STANDARD (none) -> Manufacturer Recommendations; SUPPLIER Mouser -> (none); SUPPLIER PART NUMBER 720-LST676-Q1R2-1-Z -> (none); SnapEDA_Link (none) -> https://www.snapeda.com/parts/APT2012SURCK/Kingbright/view-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
- D24: renamed from LED14; value RED -> APT2012SURCK; footprint CMAIN_PCB:LEDC2012X85N -> CMAIN_PCB:LED_APT2012SURCK; symbol Signal Distribution Box-altium-import:root_3_LED_SMD -> CMAIN_PCB:APT2012SURCK; ALTIUM_VALUE RED -> (none); Availability (none) -> In Stock; Check_prices (none) -> https://www.snapeda.com/parts/APT2012SURCK/Kingbright/view-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; MANUFACTURER (none) -> Kingbright; MAXIMUM_PACKAGE_HEIGHT (none) -> 0.75mm; MF (none) -> Kingbright; MFR ams OSRAM -> (none); MP (none) -> APT2012SURCK; MPN LS T676-Q1R2-1-Z -> (none); PARTREV (none) -> V.20B; PRICE 0.3 -> (none); Package (none) -> 0805 Kingbright; Price (none) -> None; STANDARD (none) -> Manufacturer Recommendations; SUPPLIER Mouser -> (none); SUPPLIER PART NUMBER 720-LST676-Q1R2-1-Z -> (none); SnapEDA_Link (none) -> https://www.snapeda.com/parts/APT2012SURCK/Kingbright/view-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
- D25: renamed from LED13; value RED -> APT2012SURCK; footprint CMAIN_PCB:LEDC2012X85N -> CMAIN_PCB:LED_APT2012SURCK; symbol Signal Distribution Box-altium-import:root_3_LED_SMD -> CMAIN_PCB:APT2012SURCK; ALTIUM_VALUE RED -> (none); Availability (none) -> In Stock; Check_prices (none) -> https://www.snapeda.com/parts/APT2012SURCK/Kingbright/view-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; MANUFACTURER (none) -> Kingbright; MAXIMUM_PACKAGE_HEIGHT (none) -> 0.75mm; MF (none) -> Kingbright; MFR ams OSRAM -> (none); MP (none) -> APT2012SURCK; MPN LS T676-Q1R2-1-Z -> (none); PARTREV (none) -> V.20B; PRICE 0.3 -> (none); Package (none) -> 0805 Kingbright; Price (none) -> None; STANDARD (none) -> Manufacturer Recommendations; SUPPLIER Mouser -> (none); SUPPLIER PART NUMBER 720-LST676-Q1R2-1-Z -> (none); SnapEDA_Link (none) -> https://www.snapeda.com/parts/APT2012SURCK/Kingbright/view-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
- D26: renamed from LED15; value RED -> APT2012SURCK; footprint CMAIN_PCB:LEDC2012X85N -> CMAIN_PCB:LED_APT2012SURCK; symbol Signal Distribution Box-altium-import:root_3_LED_SMD -> CMAIN_PCB:APT2012SURCK; ALTIUM_VALUE RED -> (none); Availability (none) -> In Stock; Check_prices (none) -> https://www.snapeda.com/parts/APT2012SURCK/Kingbright/view-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; MANUFACTURER (none) -> Kingbright; MAXIMUM_PACKAGE_HEIGHT (none) -> 0.75mm; MF (none) -> Kingbright; MFR ams OSRAM -> (none); MP (none) -> APT2012SURCK; MPN LS T676-Q1R2-1-Z -> (none); PARTREV (none) -> V.20B; PRICE 0.3 -> (none); Package (none) -> 0805 Kingbright; Price (none) -> None; STANDARD (none) -> Manufacturer Recommendations; SUPPLIER Mouser -> (none); SUPPLIER PART NUMBER 720-LST676-Q1R2-1-Z -> (none); SnapEDA_Link (none) -> https://www.snapeda.com/parts/APT2012SURCK/Kingbright/view-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
- D9: renamed from LED1; value RED -> APT2012SURCK; footprint CMAIN_PCB:LEDC2012X85N -> CMAIN_PCB:LED_APT2012SURCK; symbol Signal Distribution Box-altium-import:root_3_LED_SMD -> CMAIN_PCB:APT2012SURCK; ALTIUM_VALUE RED -> (none); Availability (none) -> In Stock; Check_prices (none) -> https://www.snapeda.com/parts/APT2012SURCK/Kingbright/view-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; MANUFACTURER (none) -> Kingbright; MAXIMUM_PACKAGE_HEIGHT (none) -> 0.75mm; MF (none) -> Kingbright; MFR ams OSRAM -> (none); MP (none) -> APT2012SURCK; MPN LS T676-Q1R2-1-Z -> (none); PARTREV (none) -> V.20B; PRICE 0.3 -> (none); Package (none) -> 0805 Kingbright; Price (none) -> None; STANDARD (none) -> Manufacturer Recommendations; SUPPLIER Mouser -> (none); SUPPLIER PART NUMBER 720-LST676-Q1R2-1-Z -> (none); SnapEDA_Link (none) -> https://www.snapeda.com/parts/APT2012SURCK/Kingbright/view-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
- Q4, Q5, Q6, Q7, Q8, Q9: footprint CMAIN_PCB:POWERPAK-SO-8_L5.9-W4.9-P1.27-LS6.2-BL -> CMAIN_PCB:POWERPAK-SO-8_L5.9-W4.9
