File: engineering/electronics/pcbs/CMAIN_PCB/kicad/Emergency_cutoff.kicad_sch (KiCad schematic)
At the start: 27 parts, among them K10 CPC1019N, K4 CPC1019N, K5 CPC1019N, K6 CPC1019N, K7 CPC1019N, K8 CPC1019N, K9 CPC1019N

Commit message: electronics: shorten CMAIN footprint filenames for Windows
Parts:
- R22, R26, R28, R31, R32, R39, R40, R41, R42, R43, R44, R45, R46, R47, R48, R49, R56, R57, R58, R59: footprint CMAIN_PCB:R_0805_2012Metric_Pad1.20x1.40mm_HandSolder -> CMAIN_PCB:fp_9fb50b8536
Changed lines of the file:
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@@
 			)
 		)
-		(property "Footprint" "CMAIN_PCB:R_0805_2012Metric_Pad1.20x1.40mm_HandSolder"
+		(property "Footprint" "CMAIN_PCB:fp_9fb50b8536"
 			(at 67.564 41.91 90)
 			(hide yes)
@@
 			)
 		)
-		(property "Footprint" "CMAIN_PCB:R_0805_2012Metric_Pad1.20x1.40mm_HandSolder"
+		(property "Footprint" "CMAIN_PCB:fp_9fb50b8536"
 			(at 110.49 148.59 90)
 			(hide yes)
@@
 			)
 		)
-		(property "Footprint" "CMAIN_PCB:R_0805_2012Metric_Pad1.20x1.40mm_HandSolder"
+		(property "Footprint" "CMAIN_PCB:fp_9fb50b8536"
 			(at 122.936 146.05 90)
 			(hide yes)
@@
 			)
 		)
-		(property "Footprint" "CMAIN_PCB:R_0805_2012Metric_Pad1.20x1.40mm_HandSolder"
+		(property "Footprint" "CMAIN_PCB:fp_9fb50b8536"
 			(at 186.69 90.17 90)
 			(hide yes)
@@
 			)
 		)
-		(property "Footprint" "CMAIN_PCB:R_0805_2012Metric_Pad1.20x1.40mm_HandSolder"
+		(property "Footprint" "CMAIN_PCB:fp_9fb50b8536"
 			(at 123.19 44.45 90)
 			(hide yes)
@@
 			)
 		)
-		(property "Footprint" "CMAIN_PCB:R_0805_2012Metric_Pad1.20x1.40mm_HandSolder"
+		(property "Footprint" "CMAIN_PCB:fp_9fb50b8536"
 			(at 166.37 102.87 90)
 			(hide yes)
@@
 			)
 		)
-		(property "Footprint" "CMAIN_PCB:R_0805_2012Metric_Pad1.20x1.40mm_HandSolder"
+		(property "Footprint" "CMAIN_PCB:fp_9fb50b8536"
 			(at 186.436 151.13 90)
 			(hide yes)
@@
 			)
 		)
-		(property "Footprint" "CMAIN_PCB:R_0805_2012Metric_Pad1.20x1.40mm_HandSolder"
+		(property "Footprint" "CMAIN_PCB:fp_9fb50b8536"
 			(at 166.37 44.45 90)
 			(hide yes)
@@
 			)
 		)
-		(property "Footprint" "CMAIN_PCB:R_0805_2012Metric_Pad1.20x1.40mm_HandSolder"
+		(property "Footprint" "CMAIN_PCB:fp_9fb50b8536"
 			(at 166.116 146.05 90)
 			(hide yes)
@@
 			)
 		)
-		(property "Footprint" "CMAIN_PCB:R_0805_2012Metric_Pad1.20x1.40mm_HandSolder"
+		(property "Footprint" "CMAIN_PCB:fp_9fb50b8536"
 			(at 186.69 69.85 90)
 			(hide yes)
@@
 			)
 		)
-		(property "Footprint" "CMAIN_PCB:R_0805_2012Metric_Pad1.20x1.40mm_HandSolder"
+		(property "Footprint" "CMAIN_PCB:fp_9fb50b8536"
 			(at 166.37 123.19 90)
 			(hide yes)
@@
 			)
 		)
-		(property "Footprint" "CMAIN_PCB:R_0805_2012Metric_Pad1.20x1.40mm_HandSolder"
+		(property "Footprint" "CMAIN_PCB:fp_9fb50b8536"
 			(at 186.69 107.95 90)
 			(hide yes)
@@
 			)
 		)
-		(property "Footprint" "CMAIN_PCB:R_0805_2012Metric_Pad1.20x1.40mm_HandSolder"
+		(property "Footprint" "CMAIN_PCB:fp_9fb50b8536"
 			(at 186.69 128.27 90)
 			(hide yes)
@@
 			)
 		)
-		(property "Footprint" "CMAIN_PCB:R_0805_2012Metric_Pad1.20x1.40mm_HandSolder"
+		(property "Footprint" "CMAIN_PCB:fp_9fb50b8536"
 			(at 123.19 123.19 90)
 			(hide yes)
@@
 			)
 		)
-		(property "Footprint" "CMAIN_PCB:R_0805_2012Metric_Pad1.20x1.40mm_HandSolder"
+		(property "Footprint" "CMAIN_PCB:fp_9fb50b8536"
 			(at 123.19 102.87 90)
 			(hide yes)
@@
 			)
 		)
-		(property "Footprint" "CMAIN_PCB:R_0805_2012Metric_Pad1.20x1.40mm_HandSolder"
+		(property "Footprint" "CMAIN_PCB:fp_9fb50b8536"
 			(at 166.37 85.09 90)
 			(hide yes)
@@
 			)
 		)
-		(property "Footprint" "CMAIN_PCB:R_0805_2012Metric_Pad1.20x1.40mm_HandSolder"
+		(property "Footprint" "CMAIN_PCB:fp_9fb50b8536"
 			(at 123.19 64.77 90)
 			(hide yes)
@@
 			)
 		)
-		(property "Footprint" "CMAIN_PCB:R_0805_2012Metric_Pad1.20x1.40mm_HandSolder"
+		(property "Footprint" "CMAIN_PCB:fp_9fb50b8536"
 			(at 186.69 49.53 90)
 			(hide yes)
@@
 			)
 		)
-		(property "Footprint" "CMAIN_PCB:R_0805_2012Metric_Pad1.20x1.40mm_HandSolder"
+		(property "Footprint" "CMAIN_PCB:fp_9fb50b8536"
 			(at 166.37 64.77 90)
 			(hide yes)
@@
 			)
 		)
-		(property "Footprint" "CMAIN_PCB:R_0805_2012Metric_Pad1.20x1.40mm_HandSolder"
+		(property "Footprint" "CMAIN_PCB:fp_9fb50b8536"
 			(at 123.19 85.09 90)
 			(hide yes)

Commit message: Clean up CMAIN part value fields
Parts:
- R22, R26, R42, R43, R44, R45, R46: value 1K5 -> 1K5 150V; footprint CMAIN_PCB:fp_9fb50b8536 -> Resistor_SMD:R_0805_2012Metric_Pad1.20x1.40mm_HandSolder
- R28, R31, R32, R39, R40, R41: value 1R -> 1R 150V; footprint CMAIN_PCB:fp_9fb50b8536 -> Resistor_SMD:R_0805_2012Metric_Pad1.20x1.40mm_HandSolder
- R47, R48, R49, R56, R57, R58, R59: value 47K -> 47K 150V; footprint CMAIN_PCB:fp_9fb50b8536 -> Resistor_SMD:R_0805_2012Metric_Pad1.20x1.40mm_HandSolder
Changed lines of the file:
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@@
 			)
 		)
-		(property "Value" "1K5"
+		(property "Value" "1K5 150V"
 			(at 67.564 36.83 90)
 			(show_name no)
@@
 			)
 		)
-		(property "Footprint" "CMAIN_PCB:fp_9fb50b8536"
+		(property "Footprint" "Resistor_SMD:R_0805_2012Metric_Pad1.20x1.40mm_HandSolder"
 			(at 67.564 41.91 90)
 			(hide yes)
@@
 			)
 		)
-		(property "Value" "47K"
+		(property "Value" "47K 150V"
 			(at 106.934 148.59 90)
 			(show_name no)
@@
 			)
 		)
-		(property "Footprint" "CMAIN_PCB:fp_9fb50b8536"
+		(property "Footprint" "Resistor_SMD:R_0805_2012Metric_Pad1.20x1.40mm_HandSolder"
 			(at 110.49 148.59 90)
 			(hide yes)
@@
 			)
 		)
-		(property "Value" "1K5"
+		(property "Value" "1K5 150V"
 			(at 122.936 142.494 90)
 			(show_name no)
@@
 			)
 		)
-		(property "Footprint" "CMAIN_PCB:fp_9fb50b8536"
+		(property "Footprint" "Resistor_SMD:R_0805_2012Metric_Pad1.20x1.40mm_HandSolder"
 			(at 122.936 146.05 90)
 			(hide yes)
@@
 			)
 		)
-		(property "Value" "47K"
+		(property "Value" "47K 150V"
 			(at 183.134 90.17 90)
 			(show_name no)
@@
 			)
 		)
-		(property "Footprint" "CMAIN_PCB:fp_9fb50b8536"
+		(property "Footprint" "Resistor_SMD:R_0805_2012Metric_Pad1.20x1.40mm_HandSolder"
 			(at 186.69 90.17 90)
 			(hide yes)
@@
 			)
 		)
-		(property "Value" "1K5"
+		(property "Value" "1K5 150V"
 			(at 123.19 40.894 90)
 			(show_name no)
@@
 			)
 		)
-		(property "Footprint" "CMAIN_PCB:fp_9fb50b8536"
+		(property "Footprint" "Resistor_SMD:R_0805_2012Metric_Pad1.20x1.40mm_HandSolder"
 			(at 123.19 44.45 90)
 			(hide yes)
@@
 			)
 		)
-		(property "Value" "1R"
+		(property "Value" "1R 150V"
 			(at 166.37 99.314 90)
 			(show_name no)
@@
 			)
 		)
-		(property "Footprint" "CMAIN_PCB:fp_9fb50b8536"
+		(property "Footprint" "Resistor_SMD:R_0805_2012Metric_Pad1.20x1.40mm_HandSolder"
 			(at 166.37 102.87 90)
 			(hide yes)
@@
 			)
 		)
-		(property "Value" "47K"
+		(property "Value" "47K 150V"
 			(at 182.88 151.13 90)
 			(show_name no)
@@
 			)
 		)
-		(property "Footprint" "CMAIN_PCB:fp_9fb50b8536"
+		(property "Footprint" "Resistor_SMD:R_0805_2012Metric_Pad1.20x1.40mm_HandSolder"
 			(at 186.436 151.13 90)
 			(hide yes)
@@
 			)
 		)
-		(property "Value" "1R"
+		(property "Value" "1R 150V"
 			(at 166.37 40.894 90)
 			(show_name no)
@@
 			)
 		)
-		(property "Footprint" "CMAIN_PCB:fp_9fb50b8536"
+		(property "Footprint" "Resistor_SMD:R_0805_2012Metric_Pad1.20x1.40mm_HandSolder"
 			(at 166.37 44.45 90)
 			(hide yes)
@@
 			)
 		)
-		(property "Value" "1R"
+		(property "Value" "1R 150V"
 			(at 166.116 142.494 90)
 			(show_name no)
@@
 			)
 		)
-		(property "Footprint" "CMAIN_PCB:fp_9fb50b8536"
+		(property "Footprint" "Resistor_SMD:R_0805_2012Metric_Pad1.20x1.40mm_HandSolder"
 			(at 166.116 146.05 90)
 			(hide yes)
@@
 			)
 		)
-		(property "Value" "47K"
+		(property "Value" "47K 150V"
 			(at 183.134 69.85 90)
 			(show_name no)
@@
 			)
 		)
-		(property "Footprint" "CMAIN_PCB:fp_9fb50b8536"
+		(property "Footprint" "Resistor_SMD:R_0805_2012Metric_Pad1.20x1.40mm_HandSolder"
 			(at 186.69 69.85 90)
 			(hide yes)
@@
 			)
 		)
-		(property "Value" "1R"
+		(property "Value" "1R 150V"
 			(at 166.37 119.634 90)
 			(show_name no)
@@
 			)
 		)
-		(property "Footprint" "CMAIN_PCB:fp_9fb50b8536"
+		(property "Footprint" "Resistor_SMD:R_0805_2012Metric_Pad1.20x1.40mm_HandSolder"
 			(at 166.37 123.19 90)
 			(hide yes)
@@
 			)
 		)
-		(property "Value" "47K"
+		(property "Value" "47K 150V"
 			(at 183.134 107.95 90)
 			(show_name no)
@@
 			)
 		)
-		(property "Footprint" "CMAIN_PCB:fp_9fb50b8536"
+		(property "Footprint" "Resistor_SMD:R_0805_2012Metric_Pad1.20x1.40mm_HandSolder"
 			(at 186.69 107.95 90)
 			(hide yes)
@@
 			)
 		)
-		(property "Value" "47K"
+		(property "Value" "47K 150V"
 			(at 183.134 128.27 90)
 			(show_name no)
@@
 			)
 		)
-		(property "Footprint" "CMAIN_PCB:fp_9fb50b8536"
+		(property "Footprint" "Resistor_SMD:R_0805_2012Metric_Pad1.20x1.40mm_HandSolder"
 			(at 186.69 128.27 90)
 			(hide yes)
@@
 			)
 		)
-		(property "Value" "1K5"
+		(property "Value" "1K5 150V"
 			(at 123.19 119.634 90)
 			(show_name no)
@@
 			)
 		)
-		(property "Footprint" "CMAIN_PCB:fp_9fb50b8536"
+		(property "Footprint" "Resistor_SMD:R_0805_2012Metric_Pad1.20x1.40mm_HandSolder"
 			(at 123.19 123.19 90)
 			(hide yes)
@@
 			)
 		)
-		(property "Value" "1K5"
+		(property "Value" "1K5 150V"
 			(at 123.19 99.314 90)
 			(show_name no)
@@
 			)
 		)
-		(property "Footprint" "CMAIN_PCB:fp_9fb50b8536"
+		(property "Footprint" "Resistor_SMD:R_0805_2012Metric_Pad1.20x1.40mm_HandSolder"
 			(at 123.19 102.87 90)
 			(hide yes)
@@
 			)
 		)
-		(property "Value" "1R"
+		(property "Value" "1R 150V"
 			(at 166.37 81.534 90)
 			(show_name no)
@@
 			)
 		)
-		(property "Footprint" "CMAIN_PCB:fp_9fb50b8536"
+		(property "Footprint" "Resistor_SMD:R_0805_2012Metric_Pad1.20x1.40mm_HandSolder"
 			(at 166.37 85.09 90)
 			(hide yes)
@@
 			)
 		)
-		(property "Value" "1K5"
+		(property "Value" "1K5 150V"
 			(at 123.19 61.214 90)
 			(show_name no)
@@
 			)
 		)
-		(property "Footprint" "CMAIN_PCB:fp_9fb50b8536"
+		(property "Footprint" "Resistor_SMD:R_0805_2012Metric_Pad1.20x1.40mm_HandSolder"
 			(at 123.19 64.77 90)
 			(hide yes)
@@
 			)
 		)
-		(property "Value" "47K"
+		(property "Value" "47K 150V"
 			(at 183.134 49.53 90)
 			(show_name no)
@@
 			)
 		)
-		(property "Footprint" "CMAIN_PCB:fp_9fb50b8536"
+		(property "Footprint" "Resistor_SMD:R_0805_2012Metric_Pad1.20x1.40mm_HandSolder"
 			(at 186.69 49.53 90)
 			(hide yes)
@@
 			)
 		)
-		(property "Value" "1R"
+		(property "Value" "1R 150V"
 			(at 166.37 61.214 90)
 			(show_name no)
@@
 			)
 		)
-		(property "Footprint" "CMAIN_PCB:fp_9fb50b8536"
+		(property "Footprint" "Resistor_SMD:R_0805_2012Metric_Pad1.20x1.40mm_HandSolder"
 			(at 166.37 64.77 90)
 			(hide yes)
@@
 			)
 		)
-		(property "Value" "1K5"
+		(property "Value" "1K5 150V"
 			(at 123.19 81.534 90)
 			(show_name no)
@@
 			)
 		)
-		(property "Footprint" "CMAIN_PCB:fp_9fb50b8536"
+		(property "Footprint" "Resistor_SMD:R_0805_2012Metric_Pad1.20x1.40mm_HandSolder"
 			(at 123.19 85.09 90)
 			(hide yes)

Commit message: fix(cmain): integrate prototype ordering update
Parts:
- removed R48, R49, R56, R57, R58, R59: 47K 150V, Resistor_SMD:R_0805_2012Metric_Pad1.20x1.40mm_HandSolder, symbol Device:R
